File: kicad/Ninja-qLAMP/batch01/main_2x8/filePhotoLED.kicad_sch (KiCad schematic)
At the start: 8 parts, among them U10 TLC5929, U7 SN74LVC1GU04DCKR

Commit message: sync
Parts:
- U10: footprint Package_SO:HTSSOP-24-1EP_4.4x7.8mm_P0.65mm_EP3.4x7.8mm_Mask2.4x4.68mm_ThermalVias -> DBQ24_TEX
- renumbered JJLS1 to JLS1
Connections:
- no-connect marks 1 -> 2
Changed lines of the file:
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@@
   )
   (no_connect (at 85.09 149.86))
+  (no_connect (at 114.3 116.84))
   (bus_entry (at 118.745 186.69) (size 2.54 2.54)
     (stroke (width 0) (type default) (color 0 0 0 0))
@@
     (pin "2")
   )
-  (symbol (lib_id "Ninja-qPCR:TLC5929") (at 87.63 104.14 0) (unit 2)
+  (symbol (lib_name "TLC5929_1") (lib_id "Ninja-qPCR:TLC5929") (at 87.63 104.14 0) (unit 2)
     (in_bom yes) (on_board yes) (fields_autoplaced)
     (property "Reference" "U10" (id 0) (at 104.1717 94.5925 0)
@@
       (effects (font (size 1.524 1.524)))
     )
-    (property "Footprint" "Package_SO:HTSSOP-24-1EP_4.4x7.8mm_P0.65mm_EP3.4x7.8mm_Mask2.4x4.68mm_ThermalVias" (id 2) (at 110.49 98.044 0)
+    (property "Footprint" "DBQ24_TEX" (id 2) (at 110.49 98.044 0)
       (effects (font (size 1.524 1.524)) hide)
     )
@@
     (pin "1")
     (pin "24")
+    (pin "25")
   )
   (symbol (lib_id "Ninja-qPCR:SN74LVC1G04DBVR") (at 71.12 154.94 0) (unit 1)
@@
   )
   (symbol (lib_id "Connector:Conn_01x10_Male") (at 220.98 68.58 0) (mirror y) (unit 1)
-    (in_bom yes) (on_board yes) (fields_autoplaced)
-    (property "Reference" "JLN1" (id 0) (at 220.345 54.3773 0))
-    (property "Value" "Conn_01x10_Male" (id 1) (at 220.345 57.1524 0))
+    (in_bom yes) (on_board yes)
+    (property "Reference" "JLN1" (id 0) (at 224.79 68.58 0))
+    (property "Value" "Conn_01x10_Male" (id 1) (at 229.87 71.3551 0))
     (property "Footprint" "Connector_PinSocket_2.54mm:PinSocket_1x10_P2.54mm_Vertical" (id 2) (at 220.98 68.58 0)
       (effects (font (size 1.27 1.27)) hide)
@@
   (symbol (lib_id "Connector:Conn_01x10_Male") (at 220.98 119.38 0) (mirror y) (unit 1)
     (in_bom yes) (on_board yes) (fields_autoplaced)
-    (property "Reference" "JJLS1" (id 0) (at 220.345 105.1773 0))
-    (property "Value" "Conn_01x10_Male" (id 1) (at 220.345 107.9524 0))
+    (property "Reference" "JLS1" (id 0) (at 221.6912 119.7415 0)
+      (effects (font (size 1.27 1.27)) (justify right))
+    )
+    (property "Value" "Conn_01x10_Male" (id 1) (at 221.6912 122.5166 0)
+      (effects (font (size 1.27 1.27)) (justify right))
+    )
     (property "Footprint" "Connector_PinSocket_2.54mm:PinSocket_1x10_P2.54mm_Vertical" (id 2) (at 220.98 119.38 0)
       (effects (font (size 1.27 1.27)) hide)
