File: kicad/Ninja-qLAMP/batch01/main_2x8/filePower.kicad_sch (KiCad schematic)
At the start: 40 parts, among them J1 ALI_USB, J2 Barrel_Jack_Switch, Q1 Q_NMOS_GSD, U11 IP2721, U12 TPS63710DRRR, U13 MCP1755T-3302E_DC, U14 MCP1755T-3302E_OT, U15 CJT1117-3.3, U16 CJT1117-5.0

Commit message: sync
Parts:
- L1: footprint Capacitors_SMD:C_0805 -> Capacitor_SMD:C_0805_2012Metric
