File: kicad/NinjaLite/batch01/main_2x8/filePhoto.kicad_sch (KiCad schematic)
At the start: 36 parts, among them J12 Conn_01x06_Male, J13 Conn_01x01_Male, J14 Conn_01x01_Male, J15 Conn_01x01_Male, J16 Conn_01x01_Male, J20 Conn_01x01_Male, J21 Conn_01x05_Male, J22 Conn_01x02_Male, J23 Conn_01x01_Male, J24 Conn_01x02_Male, J25 Conn_01x02_Male, J26 Conn_01x02_Male, J27 Conn_01x02_Male, U1 ADA2200ARUZ, U2 ADS1219IPWR, U3 COM1305-0.032768-EXT-T-TR, U4 LMP7717MF_NOPB

Commit message: wiring
Parts:
- J13, J16: footprint Connector_PinSocket_2.54mm:PinSocket_1x01_P2.54mm_Vertical -> Connector_PinHeader_1.27mm:PinHeader_1x01_P1.27mm_Vertical
- J14, J15: footprint Connector_PinSocket_2.54mm:PinSocket_1x01_P2.54mm_Vertical -> Connector_PinSocket_1.27mm:PinSocket_1x01_P1.27mm_Vertical
- J20, J23: footprint Connector_PinHeader_2.54mm:PinHeader_1x01_P2.54mm_Vertical -> Connector_PinHeader_1.27mm:PinHeader_1x01_P1.27mm_Vertical
- J22, J24, J25, J26, J27: footprint Connector_PinSocket_2.54mm:PinSocket_1x02_P2.54mm_Vertical -> Connector_PinHeader_1.27mm:PinHeader_1x02_P1.27mm_Vertical
Other:
- note added: "Demodulation"
Changed lines of the file:
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@@
     (effects (font (size 1.27 1.27)) (justify left bottom))
+  )
+  (text "Demodulation" (at 27.94 26.67 0)
+    (effects (font (size 2.54 2.54)) (justify left bottom))
   )
   (text "I2C Addr\n100 0000" (at 146.05 57.15 180)
@@
     (property "Reference" "J13" (id 0) (at 73.66 163.83 0))
     (property "Value" "Conn_01x01_Male" (id 1) (at 83.82 165.1 0))
-    (property "Footprint" "Connector_PinSocket_2.54mm:PinSocket_1x01_P2.54mm_Vertical" (id 2) (at 74.93 165.1 0)
+    (property "Footprint" "Connector_PinHeader_1.27mm:PinHeader_1x01_P1.27mm_Vertical" (id 2) (at 74.93 165.1 0)
       (effects (font (size 1.27 1.27)) hide)
     )
@@
     (property "Reference" "J14" (id 0) (at 73.66 166.37 0))
     (property "Value" "Conn_01x01_Male" (id 1) (at 83.82 167.64 0))
-    (property "Footprint" "Connector_PinSocket_2.54mm:PinSocket_1x01_P2.54mm_Vertical" (id 2) (at 74.93 167.64 0)
+    (property "Footprint" "Connector_PinSocket_1.27mm:PinSocket_1x01_P1.27mm_Vertical" (id 2) (at 74.93 167.64 0)
       (effects (font (size 1.27 1.27)) hide)
     )
@@
     (property "Reference" "J15" (id 0) (at 73.66 168.91 0))
     (property "Value" "Conn_01x01_Male" (id 1) (at 83.82 170.18 0))
-    (property "Footprint" "Connector_PinSocket_2.54mm:PinSocket_1x01_P2.54mm_Vertical" (id 2) (at 74.93 170.18 0)
+    (property "Footprint" "Connector_PinSocket_1.27mm:PinSocket_1x01_P1.27mm_Vertical" (id 2) (at 74.93 170.18 0)
       (effects (font (size 1.27 1.27)) hide)
     )
@@
     (property "Reference" "J16" (id 0) (at 73.66 171.45 0))
     (property "Value" "Conn_01x01_Male" (id 1) (at 83.82 172.72 0))
-    (property "Footprint" "Connector_PinSocket_2.54mm:PinSocket_1x01_P2.54mm_Vertical" (id 2) (at 74.93 172.72 0)
+    (property "Footprint" "Connector_PinHeader_1.27mm:PinHeader_1x01_P1.27mm_Vertical" (id 2) (at 74.93 172.72 0)
       (effects (font (size 1.27 1.27)) hide)
     )
@@
     (property "Reference" "J20" (id 0) (at 73.66 173.99 0))
     (property "Value" "Conn_01x01_Male" (id 1) (at 83.82 175.26 0))
-    (property "Footprint" "Connector_PinHeader_2.54mm:PinHeader_1x01_P2.54mm_Vertical" (id 2) (at 74.93 175.26 0)
+    (property "Footprint" "Connector_PinHeader_1.27mm:PinHeader_1x01_P1.27mm_Vertical" (id 2) (at 74.93 175.26 0)
       (effects (font (size 1.27 1.27)) hide)
     )
@@
     (property "Reference" "J23" (id 0) (at 74.295 161.29 0))
     (property "Value" "Conn_01x01_Male" (id 1) (at 84.455 162.56 0))
-    (property "Footprint" "Connector_PinHeader_2.54mm:PinHeader_1x01_P2.54mm_Vertical" (id 2) (at 75.565 162.56 0)
+    (property "Footprint" "Connector_PinHeader_1.27mm:PinHeader_1x01_P1.27mm_Vertical" (id 2) (at 75.565 162.56 0)
       (effects (font (size 1.27 1.27)) hide)
     )
@@
       (effects (font (size 1.27 1.27)) (justify right))
     )
-    (property "Footprint" "Connector_PinSocket_2.54mm:PinSocket_1x02_P2.54mm_Vertical" (id 2) (at 189.23 38.1 0)
+    (property "Footprint" "Connector_PinHeader_1.27mm:PinHeader_1x02_P1.27mm_Vertical" (id 2) (at 189.23 38.1 0)
       (effects (font (size 1.27 1.27)) hide)
     )
@@
     (property "Reference" "J24" (id 0) (at 178.2023 38.735 0))
     (property "Value" "Conn_01x02_Male" (id 1) (at 180.9774 38.735 0))
-    (property "Footprint" "Connector_PinSocket_2.54mm:PinSocket_1x02_P2.54mm_Vertical" (id 2) (at 182.245 38.1 0)
+    (property "Footprint" "Connector_PinHeader_1.27mm:PinHeader_1x02_P1.27mm_Vertical" (id 2) (at 182.245 38.1 0)
       (effects (font (size 1.27 1.27)) hide)
     )
@@
     (property "Reference" "J27" (id 0) (at 250.19 63.2673 0))
     (property "Value" "Conn_01x02_Male" (id 1) (at 250.19 66.0424 0))
-    (property "Footprint" "Connector_PinSocket_2.54mm:PinSocket_1x02_P2.54mm_Vertical" (id 2) (at 250.825 67.31 0)
+    (property "Footprint" "Connector_PinHeader_1.27mm:PinHeader_1x02_P1.27mm_Vertical" (id 2) (at 250.825 67.31 0)
       (effects (font (size 1.27 1.27)) hide)
     )
@@
     (property "Reference" "J26" (id 0) (at 235.9873 57.785 0))
     (property "Value" "Conn_01x02_Male" (id 1) (at 238.7624 57.785 0))
-    (property "Footprint" "Connector_PinSocket_2.54mm:PinSocket_1x02_P2.54mm_Vertical" (id 2) (at 240.03 57.15 0)
+    (property "Footprint" "Connector_PinHeader_1.27mm:PinHeader_1x02_P1.27mm_Vertical" (id 2) (at 240.03 57.15 0)
       (effects (font (size 1.27 1.27)) hide)
     )
@@
       (effects (font (size 1.27 1.27)) (justify right))
     )
-    (property "Footprint" "Connector_PinSocket_2.54mm:PinSocket_1x02_P2.54mm_Vertical" (id 2) (at 142.24 92.71 0)
-      (effects (font (size 1.27 1.27)) hide)
-    )
+    (property "Footprint" "Connector_PinHeader_1.27mm:PinHeader_1x02_P1.27mm_Vertical" (id 2) (at 142.24 92.71 0)
+      (effects (font (size 1.27 1.27)) hide)
+    )
