File: kicad/NinjaLite/batch01/main_2x8/filePhotoLED.kicad_sch (KiCad schematic)
At the start: 8 parts, among them U10 TLC5929, U7 SN74LVC1GU04DCKR

Commit message: wiring
Parts:
- U10: footprint DBQ24_TEX -> Package_SO:HTSSOP-24-1EP_4.4x7.8mm_P0.65mm_EP3.4x7.8mm_Mask2.4x4.68mm_ThermalVias
Other:
- note added: "LED"
Changed lines of the file:
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@@
     (effects (font (size 1.27 1.27)) (justify left bottom))
+  )
+  (text "LED" (at 33.02 30.48 0)
+    (effects (font (size 2.54 2.54)) (justify left bottom))
   )
   (global_label "VCC_LED" (shape input) (at 168.91 132.08 180) (fields_autoplaced)
@@
       (effects (font (size 1.524 1.524)))
     )
-    (property "Footprint" "DBQ24_TEX" (id 2) (at 110.49 98.044 0)
+    (property "Footprint" "Package_SO:HTSSOP-24-1EP_4.4x7.8mm_P0.65mm_EP3.4x7.8mm_Mask2.4x4.68mm_ThermalVias" (id 2) (at 110.49 98.044 0)
       (effects (font (size 1.524 1.524)) hide)
     )
