File: kicad/NinjaLite/batch01/main_2x8/filePhotoMUX.kicad_sch (KiCad schematic)
At the start: 3 parts, among them U18 SN74LVC1GU04DCKR, U19 CD74HC4067M96, U20 CD74HC4067M96

Commit message: wiring
Parts:
- removed U18: SN74LVC1GU04DCKR, Ninja-qPCR:SN74LVC1GU04DBVR, symbol Ninja-qPCR:SN74LVC1G04DBVR
- removed U20: CD74HC4067M96, Package_SO:SSOP-24_5.3x8.2mm_P0.65mm, symbol Ninja-qPCR:CD74HC4067M96
- added D10A1, D10B1, D11A1, D11B1, D12A1, D12B1, D13A1, D13B1, D14A1, D14B1, D15A1, D15B1, D16A1, D16B1, D1A1, D1B1, D2A1, D2B1, D3A1, D3B1, D4A1, D4B1, D5A1, D5B1, D6A1, D6B1, D7A1, D7B1, D8A1, D8B1, D9A1, D9B1: D_Photo, Diodes_SMD:D_1206, symbol Device:D_Photo
Connections:
- net MUX_SELECT is gone; now on net 3V3D: U19.15 (*E)
- net S_PD_OUT10 is gone; now on net S_PD_OUT3: U19.17 (I14)
- net S_PD_OUT12 is gone; now on net S_PD_OUT7: U19.19 (I12)
- net S_PD_OUT14 is gone; now on net S_PD_OUT11: U19.21 (I10)
- net S_PD_OUT16 is gone; now on net S_PD_OUT15: U19.23 (I8)
- net S_PD_OUT2 is gone; now on net N_PD_OUT3: U19.3 (I6)
- net S_PD_OUT4 is gone; now on net N_PD_OUT7: U19.5 (I4)
- net S_PD_OUT6 is gone; now on net N_PD_OUT11: U19.7 (I2)
- net S_PD_OUT8 is gone; now on net N_PD_OUT15: U19.9 (I0)
- net N_PD_OUT1: now also U19.2 (I7), D1B1.1 (K)
- net N_PD_OUT11: now also D6B1.1 (K)
- net N_PD_OUT13: now also U19.8 (I1), D7B1.1 (K)
- net N_PD_OUT15: now also D8B1.1 (K)
- net N_PD_OUT3: now also D2B1.1 (K)
- net N_PD_OUT5: now also U19.4 (I5), D3B1.1 (K)
- net N_PD_OUT7: now also D4B1.1 (K)
- net N_PD_OUT9: now also U19.6 (I3), D5B1.1 (K)
- net S_PD_OUT1: now also U19.16 (I15), D9B1.1 (K); no longer U19.2 (I7)
- net S_PD_OUT11: now also D14B1.1 (K); no longer U19.18 (I13)
- net S_PD_OUT13: now also U19.22 (I9), D15B1.1 (K); no longer U19.20 (I11)
- net S_PD_OUT15: now also D16B1.1 (K); no longer U19.22 (I9)
- net S_PD_OUT3: now also D10B1.1 (K); no longer U19.4 (I5)
- net S_PD_OUT5: now also U19.18 (I13), D11B1.1 (K); no longer U19.6 (I3)
- net S_PD_OUT7: now also D12B1.1 (K); no longer U19.8 (I1)
- net S_PD_OUT9: now also U19.20 (I11), D13B1.1 (K); no longer U19.16 (I15)
- new net: D13A1.1 (K), D13B1.2 (A)
- new net: D5A1.1 (K), D5B1.2 (A)
- new net: D4A1.1 (K), D4B1.2 (A)
- new net: D3A1.1 (K), D3B1.2 (A)
- new net: D9A1.1 (K), D9B1.2 (A)
- new net: D12A1.1 (K), D12B1.2 (A)
- new net: D16A1.1 (K), D16B1.2 (A)
- new net: D15A1.1 (K), D15B1.2 (A)
- new net: D1A1.1 (K), D1B1.2 (A)
- new net: D11A1.1 (K), D11B1.2 (A)
- new net: D2A1.1 (K), D2B1.2 (A)
- new net: D6A1.1 (K), D6B1.2 (A)
- new net: D10A1.1 (K), D10B1.2 (A)
- new net: D14A1.1 (K), D14B1.2 (A)
- new net: D8A1.1 (K), D8B1.2 (A)
- new net: D7A1.1 (K), D7B1.2 (A)
- new net GNDA: D10A1.2 (A), D11A1.2 (A), D12A1.2 (A), D13A1.2 (A), D14A1.2 (A), D15A1.2 (A), D16A1.2 (A), D1A1.2 (A), D2A1.2 (A), D3A1.2 (A), D4A1.2 (A), D5A1.2 (A), D6A1.2 (A), D7A1.2 (A), D8A1.2 (A), D9A1.2 (A)
- no-connect marks 1 -> 0
Other:
- note added: "Photo Diodes"
- moved on the sheet: U19A, U19B
