File: kicad/NinjaLite/batch01/main_2x8/filePower.kicad_sch (KiCad schematic)
At the start: 40 parts, among them J1 ALI_USB, J2 Barrel_Jack_Switch, Q1 Q_NMOS_GSD, U11 IP2721, U12 TPS63710DRRR, U13 MCP1755T-3302E_DC, U14 MCP1755T-3302E_OT, U15 CJT1117-3.3, U16 CJT1117-5.0

Commit message: wiring
Connections:
- net GND: now also J1.S1 (SHELD1), J1.S2 (SHELD2), J1.S3 (SHELD3), J1.S4 (SHELD4)
- net VIN: now reaches C13.1, J1.A9 (VBUS), J1.B9 (VBUS), Q1.3 (D), U11.2 (VIN)
- no-connect marks 5 -> 1
Other:
- note added: "Power"
- note added: "V(IC,SEL,SELP) must be one of them. V(IP2721|IP2721_D,High,Floating)=20 V(IP2721|IP2721_D,F,F)=15 V(IP2721|IP2721_D,Low,F)=5 V(IP2721_D,F,H)=12 V(IP2721_D,F,L)=9 V(IP2721_MAX12,H,F)=12 V(IP2721_MAX12,F,F)=9 V(IP2721_MAX12,L,F)=5"
- note removed: "USB Power Delivery"
Changed lines of the file:
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@@
   (junction (at 102.87 147.32) (diameter 0) (color 0 0 0 0)
   )
+  (junction (at 19.05 66.04) (diameter 0) (color 0 0 0 0)
+  )
   (junction (at 102.87 149.86) (diameter 0) (color 0 0 0 0)
   )
@@
   (junction (at 124.46 80.01) (diameter 0) (color 0 0 0 0)
   )
+  (junction (at 19.05 71.12) (diameter 0) (color 0 0 0 0)
+  )
   (junction (at 248.92 123.19) (diameter 0) (color 0 0 0 0)
   )
@@
   (junction (at 154.94 171.45) (diameter 0) (color 0 0 0 0)
   )
+  (junction (at 19.05 68.58) (diameter 0) (color 0 0 0 0)
+  )
   (junction (at 217.17 93.98) (diameter 0) (color 0 0 0 0)
   )
   (junction (at 45.72 71.12) (diameter 0) (color 0 0 0 0)
   )
+  (junction (at 45.72 44.45) (diameter 0) (color 0 0 0 0)
+  )
   (junction (at 251.46 67.31) (diameter 0) (color 0 0 0 0)
   )
@@
   (junction (at 53.34 78.74) (diameter 0) (color 0 0 0 0)
   )
-  (no_connect (at 21.59 63.5))
-  (no_connect (at 21.59 66.04))
-  (no_connect (at 21.59 68.58))
-  (no_connect (at 21.59 71.12))
   (no_connect (at 59.69 139.7))
   (wire (pts (xy 66.04 58.42) (xy 63.5 58.42))
@@
     (stroke (width 0) (type default) (color 0 0 0 0))
   )
+  (wire (pts (xy 19.05 66.04) (xy 19.05 68.58))
+    (stroke (width 0) (type default) (color 0 0 0 0))
+  )
   (wire (pts (xy 220.98 125.73) (xy 220.98 128.27))
     (stroke (width 0) (type default) (color 0 0 0 0))
@@
     (stroke (width 0) (type default) (color 0 0 0 0))
   )
+  (wire (pts (xy 19.05 68.58) (xy 21.59 68.58))
+    (stroke (width 0) (type default) (color 0 0 0 0))
+  )
   (wire (pts (xy 154.94 171.45) (xy 160.02 171.45))
     (stroke (width 0) (type default) (color 0 0 0 0))
@@
     (stroke (width 0) (type default) (color 0 0 0 0))
   )
+  (wire (pts (xy 19.05 63.5) (xy 19.05 66.04))
+    (stroke (width 0) (type default) (color 0 0 0 0))
+  )
   (wire (pts (xy 190.5 59.69) (xy 190.5 66.04))
     (stroke (width 0) (type default) (color 0 0 0 0))
@@
     (stroke (width 0) (type default) (color 0 0 0 0))
   )
+  (wire (pts (xy 19.05 71.12) (xy 21.59 71.12))
+    (stroke (width 0) (type default) (color 0 0 0 0))
+  )
+  (wire (pts (xy 43.18 44.45) (xy 45.72 44.45))
+    (stroke (width 0) (type default) (color 0 0 0 0))
+  )
   (wire (pts (xy 223.52 93.98) (xy 217.17 93.98))
     (stroke (width 0) (type default) (color 0 0 0 0))
@@
     (stroke (width 0) (type default) (color 0 0 0 0))
   )
+  (wire (pts (xy 21.59 63.5) (xy 19.05 63.5))
+    (stroke (width 0) (type default) (color 0 0 0 0))
+  )
   (wire (pts (xy 102.87 113.03) (xy 102.87 115.57))
     (stroke (width 0) (type default) (color 0 0 0 0))
@@
     (stroke (width 0) (type default) (color 0 0 0 0))
   )
+  (wire (pts (xy 19.05 68.58) (xy 19.05 71.12))
+    (stroke (width 0) (type default) (color 0 0 0 0))
+  )
   (wire (pts (xy 175.26 93.98) (xy 185.42 93.98))
     (stroke (width 0) (type default) (color 0 0 0 0))
@@
     (stroke (width 0) (type default) (color 0 0 0 0))
   )
+  (wire (pts (xy 19.05 71.12) (xy 19.05 80.01))
+    (stroke (width 0) (type default) (color 0 0 0 0))
+  )
   (wire (pts (xy 196.85 107.95) (xy 196.85 111.76))
     (stroke (width 0) (type default) (color 0 0 0 0))
   )
+  (wire (pts (xy 19.05 66.04) (xy 21.59 66.04))
+    (stroke (width 0) (type default) (color 0 0 0 0))
+  )
   (wire (pts (xy 97.79 149.86) (xy 102.87 149.86))
     (stroke (width 0) (type default) (color 0 0 0 0))
@@
     (stroke (width 0) (type default) (color 0 0 0 0))
   )
-  (text "USB Power Delivery" (at 22.86 31.75 0)
+  (text "V(IC,SEL,SELP) must be one of them.\nV(IP2721|IP2721_D,High,Floating)=20\nV(IP2721|IP2721_D,F,F)=15\nV(IP2721|IP2721_D,Low,F)=5\nV(IP2721_D,F,H)=12\nV(IP2721_D,F,L)=9\nV(IP2721_MAX12,H,F)=12\nV(IP2721_MAX12,F,F)=9\nV(IP2721_MAX12,L,F)=5"
+    (at 113.03 107.95 0)
+    (effects (font (size 1.27 1.27)) (justify left bottom))
+  )
+  (text "Power" (at 22.86 31.75 0)
     (effects (font (size 2.54 2.54)) (justify left bottom))
   )
@@
       (effects (font (size 1.27 1.27)) hide)
     )
+  )
+  (hierarchical_label "VIN" (shape input) (at 43.18 44.45 180)
+    (effects (font (size 1.27 1.27)) (justify right))
   )
   (hierarchical_label "SELP" (shape input) (at 88.9 63.5 0)
@@
       (effects (font (size 1.27 1.27)) hide)
     )
+    (pin "1")
+  )
+  (symbol (lib_id "power:GND") (at 19.05 80.01 0) (unit 1)
+    (in_bom yes) (on_board yes)
+    (property "Reference" "#PWR0105" (id 0) (at 19.05 86.36 0)
+      (effects (font (size 1.27 1.27)) hide)
+    )
+    (property "Value" "GND" (id 1) (at 19.177 84.4042 0))
+    (property "Footprint" "" (id 2) (at 19.05 80.01 0)
+      (effects (font (size 1.27 1.27)) hide)
+    )
+    (property "Datasheet" "" (id 3) (at 19.05 80.01 0)
+      (effects (font (size 1.27 1.27)) hide)
+    )
