File: kicad/NinjaLite/batch01/main_2x8/filePhotoThermistors.kicad_sch (KiCad schematic)
At the start: 11 parts, among them J28 Conn_01x09_Male, U8 TS12A12511DCNR, U9 CD74HC4067M96

Commit message: wiring
Parts:
- removed J28: Conn_01x09_Male, Connector_PinSocket_1.27mm:PinSocket_1x09_P1.27mm_Vertical, symbol Connector:Conn_01x09_Male
- removed U9: CD74HC4067M96, Package_SO:SSOP-24_5.3x8.2mm_P0.65mm, symbol Ninja-qPCR:CD74HC4067M96
- added U9: SN74LV4051A, Package_SO:SOIC-16_3.9x9.9mm_P1.27mm, symbol Ninja-qPCR:SN74LV4051A
Connections:
- net 3V3D: now also U9.16 (VCC)
- net GND: now also U9.6 (INH), U9.7 (GND), U9.8 (GND)
- net MUX_S0: now also U9.11 (A)
- net MUX_S1: now also U9.10 (B)
- net MUX_S2: now also U9.9 (C)
- net THERM_AIR: now also U9.14 (Y1)
- net THERM_EXT1: now also U9.12 (Y3)
- net THERM_EXT2: now also U9.1 (Y4)
- net THERM_EXT3: now also U9.5 (Y5)
- net THERM_LID: now also U9.15 (Y2)
- net THERM_MUX_OUT: now also U9.3 (COM)
- net THERM_WELL: now also U9.13 (Y0)
- no-connect marks 0 -> 5
Other:
- note added: "Thermistors"
