File: kicad/NinjaLite/batch01/main_2x8/qLAMP-main.kicad_pcb (KiCad board)
At the start: 2 copper layers, 223.1 x 116 mm, 147 parts, among them J1 ALI_USB, J12 Conn_01x06_Male, J13 Conn_01x01_Male, J14 Conn_01x01_Male, J15 Conn_01x01_Male, J16 Conn_01x01_Male, J2 Barrel_Jack_Switch, J20 Conn_01x01_Male, J21 Conn_01x05_Male, J22 Conn_01x02_Male, J23 Conn_01x01_Male, J24 Conn_01x02_Male, J25 Conn_01x02_Male, J26 Conn_01x02_Male, J27 Conn_01x02_Male, J28 Conn_01x09_Male, Q1 Q_NMOS_GSD, Q3 Q_NMOS_GSD, Q5 Q_NMOS_GSD, U1 ADA2200ARUZ, U10 TLC5929, U11 IP2721, U12 TPS63710DRRR, U13 MCP1755T-3302E_DC, U14 MCP1755T-3302E_OT, U15 CJT1117-3.3, U16 CJT1117-5.0, U17 LITE_LCD, U18 SN74LVC1GU04DCKR, U19 CD74HC4067M96, U2 ADS1219IPWR, U20 CD74HC4067M96, U3 COM1305-0.032768-EXT-T-TR, U4 LMP7717MF_NOPB, U5 ESP32-WROOM-32, U6 ESP32-WROOM-32U, U7 SN74LVC1GU04DCKR, U8 TS12A12511DCNR, U9 CD74HC4067M96

Commit message: renmaed
Parts:
- moved U20 149.6 mm to (33.5, 94.7), turned to 90 degrees
- moved C27 134.3 mm to (72.5, 162.0)
- moved C5 134.3 mm to (45.4, 168.2)
- moved J15 134.3 mm to (46.1, 171.0)
- moved J16 134.3 mm to (43.5, 148.4)
- moved J22 134.3 mm to (43.5, 163.6)
- moved J26 134.3 mm to (43.5, 150.9)
- moved J27 134.3 mm to (43.5, 156.0)
- moved JP4 134.3 mm to (44.9, 166.3)
- moved JP5 134.3 mm to (44.9, 168.5)
- moved JP7 134.3 mm to (49.9, 151.5)
- moved R14 134.3 mm to (52.7, 164.4)
- moved R15 134.3 mm to (76.9, 149.5)
- moved R16 134.3 mm to (66.7, 151.2)
- moved U18 134.3 mm to (57.3, 152.5)
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
Commit message: wiring
Parts:
- removed J28: Conn_01x09_Male, Connector_PinSocket_1.27mm:PinSocket_1x09_P1.27mm_Vertical
- removed JP2, JP3: Jumper_2_Bridged, Jumper:SolderJumper-2_P1.3mm_Open_TrianglePad1.0x1.5mm
- removed SERIAL4: Conn_01x04_Male, Connector_PinSocket_2.54mm:PinSocket_1x04_P2.54mm_Vertical
- removed SERIAL6: Conn_01x06_Male, Connector_PinSocket_2.54mm:PinSocket_1x06_P2.54mm_Vertical
- removed U18: SN74LVC1GU04DCKR, Ninja-qPCR:SN74LVC1GU04DBVR
- removed U20: CD74HC4067M96, Package_SO:SSOP-24_5.3x8.2mm_P0.65mm
- removed U6: ESP32-WROOM-32U, RF_Module:ESP32-WROOM-32U
- added J3: Conn_01x06_Male, Connector_PinHeader_2.54mm:PinHeader_1x06_P2.54mm_Vertical, F.Cu at (159.7, 122.3)
- added R21: 100k, Resistor_SMD:R_0603_1608Metric, F.Cu at (150.4, 119.4)
- added R22: 100k, Resistor_SMD:R_0603_1608Metric, F.Cu at (147.3, 119.4)
- added R23: 100k, Resistor_SMD:R_0603_1608Metric, F.Cu at (153.4, 119.4)
- C9: value 0.1uF -> 10uF; footprint Capacitor_SMD:C_0603_1608Metric -> Capacitor_SMD:C_0805_2012Metric
- J13, J16: footprint Connector_PinSocket_2.54mm:PinSocket_1x01_P2.54mm_Vertical -> Connector_PinHeader_1.27mm:PinHeader_1x01_P1.27mm_Vertical
- J14, J15: footprint Connector_PinSocket_2.54mm:PinSocket_1x01_P2.54mm_Vertical -> Connector_PinSocket_1.27mm:PinSocket_1x01_P1.27mm_Vertical
- J20, J23: footprint Connector_PinHeader_2.54mm:PinHeader_1x01_P2.54mm_Vertical -> Connector_PinHeader_1.27mm:PinHeader_1x01_P1.27mm_Vertical
- J22, J24, J25, J26, J27: footprint Connector_PinSocket_2.54mm:PinSocket_1x02_P2.54mm_Vertical -> Connector_PinHeader_1.27mm:PinHeader_1x02_P1.27mm_Vertical
- JP10, JP8, JP9: moved to B.Cu
- R1: value 10k -> 100k
- U9: value CD74HC4067M96 -> SN74LV4051A; footprint Package_SO:SSOP-24_5.3x8.2mm_P0.65mm -> Package_SO:SOIC-16_3.9x9.9mm_P1.27mm
- moved C31 159.6 mm to (221.7, 109.0)
- moved C29 148.1 mm to (209.0, 106.4)
- moved C20 131.7 mm to (94.2, 95.2), turned to 90 degrees
- moved C27 128.7 mm to (173.7, 82.6), turned to 90 degrees
- moved C19 120.3 mm to (97.8, 98.2), turned to 180 degrees
- moved JP8 114.4 mm to (122.5, 112.7), turned to 180 degrees
- moved U17 114.0 mm to (115.9, 89.2)
- moved R16 105.2 mm to (139.8, 75.5), turned to 0 degrees
- moved C30 104.9 mm to (76.5, 91.3), turned to 90 degrees
- moved R17 101.3 mm to (120.7, 90.1), turned to 0 degrees
- moved U5 99.6 mm to (150.8, 103.4), turned to -90 degrees
- moved C33 99.4 mm to (74.4, 91.3), turned to 90 degrees
- moved R18 98.2 mm to (117.3, 90.1), turned to 180 degrees
- moved C26 95.2 mm to (78.2, 91.3)
- moved R5 94.7 mm to (98.7, 91.0), turned to 180 degrees
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Connections:
- net Net-(C13-Pad1) renamed /Power/VIN
- net S_PD_OUT16 renamed /PhotoMUX/S_PD_OUT15
- C9 pad 1: /EN -> Net-(C9-Pad1)
- D10A1 pad 1: S_PD_OUT3 -> Net-(D10A1-Pad1)
- D10B1 pad 1: S_PD_OUT4 -> /PhotoMUX/S_PD_OUT3
- D10B1 pad 2: GNDA -> Net-(D10A1-Pad1)
- D11A1 pad 1: S_PD_OUT5 -> Net-(D11A1-Pad1)
- D11B1 pad 1: S_PD_OUT6 -> /PhotoMUX/S_PD_OUT5
- D11B1 pad 2: GNDA -> Net-(D11A1-Pad1)
- D12A1 pad 1: S_PD_OUT7 -> Net-(D12A1-Pad1)
- D12B1 pad 1: S_PD_OUT8 -> /PhotoMUX/S_PD_OUT7
- D12B1 pad 2: GNDA -> Net-(D12A1-Pad1)
- D13A1 pad 1: S_PD_OUT9 -> Net-(D13A1-Pad1)
- D13B1 pad 1: S_PD_OUT10 -> /PhotoMUX/S_PD_OUT9
- D13B1 pad 2: GNDA -> Net-(D13A1-Pad1)
- D14A1 pad 1: S_PD_OUT11 -> Net-(D14A1-Pad1)
- D14B1 pad 1: S_PD_OUT12 -> /PhotoMUX/S_PD_OUT11
- D14B1 pad 2: GNDA -> Net-(D14A1-Pad1)
- D15A1 pad 1: S_PD_OUT13 -> Net-(D15A1-Pad1)
- D15B1 pad 1: S_PD_OUT14 -> /PhotoMUX/S_PD_OUT13
- D15B1 pad 2: GNDA -> Net-(D15A1-Pad1)
- D16A1 pad 1: S_PD_OUT15 -> Net-(D16A1-Pad1)
- D16B1 pad 2: GNDA -> Net-(D16A1-Pad1)
- D1A1 pad 1: N_PD_OUT1 -> Net-(D1A1-Pad1)
- D1B1 pad 1: N_PD_OUT2 -> /PhotoMUX/N_PD_OUT1
- D1B1 pad 2: GNDA -> Net-(D1A1-Pad1)
- D2A1 pad 1: N_PD_OUT3 -> Net-(D2A1-Pad1)
- D2B1 pad 1: N_PD_OUT4 -> /PhotoMUX/N_PD_OUT3
- D2B1 pad 2: GNDA -> Net-(D2A1-Pad1)
- D3A1 pad 1: N_PD_OUT5 -> Net-(D3A1-Pad1)
- D3B1 pad 1: N_PD_OUT6 -> /PhotoMUX/N_PD_OUT5
- D3B1 pad 2: GNDA -> Net-(D3A1-Pad1)
- D4A1 pad 1: N_PD_OUT7 -> Net-(D4A1-Pad1)
- D4B1 pad 1: N_PD_OUT8 -> /PhotoMUX/N_PD_OUT7
- D4B1 pad 2: GNDA -> Net-(D4A1-Pad1)
- D5A1 pad 1: N_PD_OUT9 -> Net-(D5A1-Pad1)
- D5B1 pad 1: N_PD_OUT10 -> /PhotoMUX/N_PD_OUT9
- D5B1 pad 2: GNDA -> Net-(D5A1-Pad1)
- D6A1 pad 1: N_PD_OUT11 -> Net-(D6A1-Pad1)
- D6B1 pad 1: N_PD_OUT12 -> /PhotoMUX/N_PD_OUT11
- D6B1 pad 2: GNDA -> Net-(D6A1-Pad1)
- D7A1 pad 1: N_PD_OUT13 -> Net-(D7A1-Pad1)
- D7B1 pad 1: N_PD_OUT14 -> /PhotoMUX/N_PD_OUT13
- D7B1 pad 2: GNDA -> Net-(D7A1-Pad1)
- D8A1 pad 1: N_PD_OUT15 -> Net-(D8A1-Pad1)
- D8B1 pad 1: N_PD_OUT16 -> /PhotoMUX/N_PD_OUT15
- D8B1 pad 2: GNDA -> Net-(D8A1-Pad1)
- D9A1 pad 1: S_PD_OUT1 -> Net-(D9A1-Pad1)
- D9B1 pad 1: S_PD_OUT2 -> /PhotoMUX/S_PD_OUT1
- D9B1 pad 2: GNDA -> Net-(D9A1-Pad1)
- J1 pad S1: unconnected-(J1-PadS1) -> GNDD
- J1 pad S2: unconnected-(J1-PadS2) -> GNDD
- J1 pad S3: unconnected-(J1-PadS3) -> GNDD
- J1 pad S4: unconnected-(J1-PadS4) -> GNDD
- R1 pad 1: 3V3D -> Net-(C9-Pad1)
- R1 pad 2: /EN -> 3V3D
- U19 pad 15: MUX_SELECT -> 3V3D
- U19 pad 16: S_PD_OUT9 -> /PhotoMUX/S_PD_OUT1
- U19 pad 17: S_PD_OUT10 -> /PhotoMUX/S_PD_OUT3
- U19 pad 18: S_PD_OUT11 -> /PhotoMUX/S_PD_OUT5
- U19 pad 19: S_PD_OUT12 -> /PhotoMUX/S_PD_OUT7
- U19 pad 2: S_PD_OUT1 -> /PhotoMUX/N_PD_OUT1
- U19 pad 20: S_PD_OUT13 -> /PhotoMUX/S_PD_OUT9
- U19 pad 21: S_PD_OUT14 -> /PhotoMUX/S_PD_OUT11
- U19 pad 22: S_PD_OUT15 -> /PhotoMUX/S_PD_OUT13
- U19 pad 3: S_PD_OUT2 -> /PhotoMUX/N_PD_OUT3
- U19 pad 4: S_PD_OUT3 -> /PhotoMUX/N_PD_OUT5
- U19 pad 5: S_PD_OUT4 -> /PhotoMUX/N_PD_OUT7
- U19 pad 6: S_PD_OUT5 -> /PhotoMUX/N_PD_OUT9
- U19 pad 7: S_PD_OUT6 -> /PhotoMUX/N_PD_OUT11
- U19 pad 8: S_PD_OUT7 -> /PhotoMUX/N_PD_OUT13
- U19 pad 9: S_PD_OUT8 -> /PhotoMUX/N_PD_OUT15
- U5 pad 10: unconnected-(U5-Pad10) -> LED_G
- U5 pad 11: unconnected-(U5-Pad11) -> LED_B
- U5 pad 12: unconnected-(U5-Pad12) -> THERM_R_SWITCH
- U5 pad 13: unconnected-(U5-Pad13) -> LED_LAT
- U5 pad 14: unconnected-(U5-Pad14) -> LED_SPI_SCLK
- U5 pad 16: unconnected-(U5-Pad16) -> LED_SPI_MOSI
- U5 pad 23: unconnected-(U5-Pad23) -> LED_SPI_MISO
- U5 pad 24: unconnected-(U5-Pad24) -> TACT3
- U5 pad 25: unconnected-(U5-Pad25) -> TACT2
- U5 pad 26: unconnected-(U5-Pad26) -> TACT1
- U5 pad 28: unconnected-(U5-Pad28) -> ADC_DRDY
- U5 pad 29: unconnected-(U5-Pad29) -> I2C_SDA
- U5 pad 3: /EN -> Net-(C9-Pad1)
- U5 pad 30: unconnected-(U5-Pad30) -> I2C_SCL
- U5 pad 31: unconnected-(U5-Pad31) -> MUX_S0
- U5 pad 33: unconnected-(U5-Pad33) -> MUX_S1
- U5 pad 34: unconnected-(U5-Pad34) -> /RXD
- U5 pad 35: unconnected-(U5-Pad35) -> /TXD
- U5 pad 36: unconnected-(U5-Pad36) -> MUX_S2
- U5 pad 37: unconnected-(U5-Pad37) -> MUX_S3
- U5 pad 6: unconnected-(U5-Pad6) -> VIN_SENSE
- U5 pad 7: unconnected-(U5-Pad7) -> /LID_HEATER
- U5 pad 8: unconnected-(U5-Pad8) -> /WELL_HEATER
- U5 pad 9: unconnected-(U5-Pad9) -> LED_R
- U9 pad 1: THERM_MUX_OUT -> THERM_EXT2
- U9 pad 10: MUX_S0 -> MUX_S1
- U9 pad 11: MUX_S1 -> MUX_S0
- U9 pad 12: GNDD -> THERM_EXT1
- U9 pad 13: MUX_S3 -> THERM_WELL
- U9 pad 14: MUX_S2 -> THERM_AIR
- U9 pad 15: 3V3D -> THERM_LID
- U9 pad 16: THERM_EXT11 -> 3V3D
- U9 pad 2: PD_TH2 -> unconnected-(U9-Pad2)
- U9 pad 3: PD_TH1 -> THERM_MUX_OUT
- U9 pad 4: THERM_EXT3 -> unconnected-(U9-Pad4)
- U9 pad 5: THERM_EXT2 -> THERM_EXT3
- U9 pad 6: THERM_EXT1 -> GNDD
- U9 pad 7: THERM_LID -> GNDD
- U9 pad 8: THERM_AIR -> GNDD
- U9 pad 9: THERM_WELL -> MUX_S2
Routing:
- net GNDD: track 0.00 -> 387.9 mm, vias 0 -> 14
- net 3V3D: track 0.00 -> 290.1 mm, vias 0 -> 11
- net GNDA: track 0.00 -> 262.5 mm, vias 0 -> 21
- net MUX_S1: track 0.00 -> 191.3 mm, vias 0 -> 3
- net MUX_S0: track 0.00 -> 185.0 mm, vias 0 -> 3
- net 12V: track 0.00 -> 183.8 mm, vias 0 -> 1
- net MUX_S2: track 0.00 -> 178.3 mm, vias 0 -> 3
- net MUX_S3: track 0.00 -> 158.8 mm, vias 0 -> 2
- net THERM_MUX_OUT: track 0.00 -> 125.1 mm, vias 0 -> 6
- net /PhotoMUX/N_PD_OUT1: track 0.00 -> 124.2 mm
- net /PhotoMUX/N_PD_OUT3: track 0.00 -> 113.2 mm
- net /PhotoMUX/S_PD_OUT1: track 0.00 -> 111.9 mm
- net I2C_SCL: track 0.00 -> 108.4 mm, vias 0 -> 4
- net I2C_SDA: track 0.00 -> 106.2 mm, vias 0 -> 4
- net ADC_DRDY: track 0.00 -> 104.8 mm, vias 0 -> 4
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- added copper zone on F.Cu, net 3V3D
Other:
- board size 223.1 x 116 mm -> 159.2 x 58 mm
- board text added: "NinjaLite"
- board text removed: "*"
- board text removed: "+"
- board text removed: "12"
- board text removed: "12V"
- board text removed: "12V_UPS"
- board text removed: "13"
- board text removed: "14"
- board text removed: "150*5"
- board text removed: "2.1mm DCJack Center+"
- board text removed: "22"
- board text removed: "3"
- board text removed: "47k*7"
- board text removed: "4Pin DIN"
- board text removed: "5"
- board text removed: "5V_UPS"
- board text removed: "7"
- board text removed: "BLACK"
- board text removed: "DOOR"
- board text removed: "EPS12V"
- board text removed: "FAN"
- board text removed: "GBAR"
- board text removed: "GND"
- board text removed: "GPIO29"
- board text removed: "LOCK"
- board text removed: "Ninja Lite"
- board text removed: "PELTIER"
- board text removed: "RED"
- board text removed: "UPS"
- board text removed: "batch16/photo-dual"

Commit message: sync
Parts:
- moved R16 49.0 mm to (187.5, 86.8), turned to -90 degrees
- moved TAIR1 48.5 mm to (163.6, 90.6)
- moved TLID1 48.5 mm to (159.6, 90.6)
- moved TWELL1 48.5 mm to (167.6, 90.6)
- moved JP10 48.2 mm to (189.1, 82.4), turned to 90 degrees
- moved R4 48.1 mm to (187.5, 83.8)
- moved C31 46.6 mm to (175.3, 113.4)
- moved C28 46.6 mm to (175.2, 110.6)
- moved R3 46.3 mm to (187.5, 80.7)
- moved JP9 45.7 mm to (187.0, 82.4), turned to 90 degrees
- moved R18 43.8 mm to (160.6, 97.1)
- moved R17 43.8 mm to (163.9, 97.1)
- moved J2 42.8 mm to (204.3, 85.8)
- moved JLS1 42.8 mm to (186.0, 126.6)
- moved JP1 42.8 mm to (152.6, 128.8)
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Connections:
- U5 pad 6: VIN_SENSE -> /WELL_HEATER
- U5 pad 8: /WELL_HEATER -> VIN_SENSE
Routing:
- net GNDD: track 387.9 -> 561.5 mm, vias 14 -> 27
- net 5V: track 31.4 -> 84.7 mm, vias 0 -> 1
- net I2C_SCL: track 108.4 -> 152.6 mm
- net VIN_SENSE: track 0.00 -> 43.4 mm, vias 0 -> 2
- net I2C_SDA: track 106.2 -> 149.2 mm, vias 4 -> 5
- net 3V3D: track 290.1 -> 322.5 mm, vias 11 -> 17
- net LED_R: track 8.51 -> 39.1 mm, vias 0 -> 2
- net LED_G: track 11.4 -> 40.7 mm, vias 0 -> 2
- net LED_B: track 13.6 -> 41.8 mm, vias 0 -> 2
- net /LID_HEATER: track 0.00 -> 22.7 mm
- net 12V: track 183.8 -> 168.8 mm, vias 1 -> 2
- net /WELL_HEATER: track 0.00 -> 13.4 mm
- net TACT1: track 13.9 -> 25.8 mm
- net /Power/SEL: track 0.00 -> 11.0 mm, vias 0 -> 1
- net /PhotoLED/N_LED_OUT7: track 46.3 -> 37.0 mm
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Other:
- board size 159.2 x 58 mm -> 142 x 58 mm
- board text added: "batch01/main"
- board text removed: "batch01/main_2x8"
