File: kicad/NinjaLite/batch01/main/filePhotoLED.kicad_sch (KiCad schematic)
At the start: 8 parts, among them U10 TLC5929, U7 SN74LVC1GU04DCKR

Commit message: dru cleared
Parts:
- JLN1, JLS1: footprint Connector_PinSocket_2.54mm:PinSocket_1x10_P2.54mm_Vertical -> Connector_PinHeader_2.54mm:PinHeader_1x10_P2.54mm_Vertical
Changed lines of the file:
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@@
     (property "Reference" "JLN1" (id 0) (at 224.79 68.58 0))
     (property "Value" "Conn_01x10_Male" (id 1) (at 229.87 71.3551 0))
-    (property "Footprint" "Connector_PinSocket_2.54mm:PinSocket_1x10_P2.54mm_Vertical" (id 2) (at 220.98 68.58 0)
+    (property "Footprint" "Connector_PinHeader_2.54mm:PinHeader_1x10_P2.54mm_Vertical" (id 2) (at 220.98 68.58 0)
       (effects (font (size 1.27 1.27)) hide)
     )
@@
       (effects (font (size 1.27 1.27)) (justify right))
     )
-    (property "Footprint" "Connector_PinSocket_2.54mm:PinSocket_1x10_P2.54mm_Vertical" (id 2) (at 220.98 119.38 0)
+    (property "Footprint" "Connector_PinHeader_2.54mm:PinHeader_1x10_P2.54mm_Vertical" (id 2) (at 220.98 119.38 0)
       (effects (font (size 1.27 1.27)) hide)
     )
