File: kicad/NinjaLite/batch01/main/qLAMP-main.kicad_sch (KiCad schematic)
At the start: 16 parts, among them J3 Conn_01x06_Male, Q3 Q_NMOS_GSD, Q5 Q_NMOS_GSD, U17 LITE_LCD, U5 ESP32-WROOM-32

Commit message: dru cleared
Connections:
- net GND: now also J3.1 (Pin_1); no longer J3.3 (Pin_3)
- net RXD: now also J3.4 (Pin_4); no longer J3.2 (Pin_2)
- net TACT2: now also J3.2 (Pin_2); no longer J3.6 (Pin_6)
- net TXD: now also J3.3 (Pin_3); no longer J3.1 (Pin_1)
- net VCCL renamed 5V
