File: kicad/NinjaLite/batch01/main/qLAMP-main.kicad_pcb (KiCad board)
At the start: 2 copper layers, 142 x 58 mm, 143 parts, among them J1 ALI_USB, J12 Conn_01x06_Male, J13 Conn_01x01_Male, J14 Conn_01x01_Male, J15 Conn_01x01_Male, J16 Conn_01x01_Male, J2 Barrel_Jack_Switch, J20 Conn_01x01_Male, J21 Conn_01x05_Male, J22 Conn_01x02_Male, J23 Conn_01x01_Male, J24 Conn_01x02_Male, J25 Conn_01x02_Male, J26 Conn_01x02_Male, J27 Conn_01x02_Male, J3 Conn_01x06_Male, Q1 Q_NMOS_GSD, Q3 Q_NMOS_GSD, Q5 Q_NMOS_GSD, U1 ADA2200ARUZ, U10 TLC5929, U11 IP2721, U12 TPS63710DRRR, U13 MCP1755T-3302E_DC, U14 MCP1755T-3302E_OT, U15 CJT1117-3.3, U16 CJT1117-5.0, U17 LITE_LCD, U19 CD74HC4067M96, U2 ADS1219IPWR, U3 COM1305-0.032768-EXT-T-TR, U4 LMP7717MF_NOPB, U5 ESP32-WROOM-32, U7 SN74LVC1GU04DCKR, U8 TS12A12511DCNR, U9 SN74LV4051A

Commit message: dru cleared
Parts:
- JLN1, JLS1: footprint Connector_PinSocket_2.54mm:PinSocket_1x10_P2.54mm_Vertical -> Connector_PinHeader_2.54mm:PinHeader_1x10_P2.54mm_Vertical
- moved C2 0.89 mm to (97.9, 99.2), turned to 180 degrees
Connections:
- J3 pad 1: /TXD -> GNDD
- J3 pad 2: /RXD -> TACT2
- J3 pad 3: GNDD -> /TXD
- J3 pad 4: unconnected-(J3-Pad4) -> /RXD
- J3 pad 6: TACT2 -> unconnected-(J3-Pad6)
- U17 pad 9: VCCL -> 5V
Routing:
- net TACT2: track 18.6 -> 34.3 mm, vias 0 -> 1
- net 5V: track 84.7 -> 99.1 mm
- net GNDD: track 561.5 -> 569.1 mm
- net VCCL: track 5.80 -> 0.00 mm, vias 1 -> 0
- net TACT1: track 25.8 -> 21.5 mm
- net /TXD: track 11.8 -> 8.21 mm
- net GNDA: track 269.7 -> 266.5 mm, vias 21 -> 20
- net 12V: track 168.8 -> 171.5 mm
- net /Photo/ADA8: track 6.58 -> 4.71 mm
- net /RXD: track 10.3 -> 8.76 mm
- net /Photo/PN2: track 24.2 -> 23.4 mm
Other:
- outline, holes or cut-outs redrawn

Commit message: just before placing vias
Parts:
- moved JP1 6.30 mm to (147.0, 126.0)
- moved JP4 0.37 mm to (98.5, 99.3)
- moved JP5 0.37 mm to (98.5, 102.0)
Routing:
- net GNDA: track 266.5 -> 259.3 mm
- net /Photo/PP1: track 26.5 -> 25.7 mm
- net GNDD: track 569.1 -> 569.7 mm
- added copper zone on F.Cu, net -1V
- added copper zone on F.Cu, net /Power/VIN
- added copper zone on F.Cu, net 12V
- added copper zone on B.Cu, net GNDA
- added copper zone on F.Cu, net GNDA
- added copper zone on B.Cu, net GNDD
- added copper zone on F.Cu, net GNDD
Other:
- outline, holes or cut-outs redrawn
- board text added: "*"
- board text added: "GND"
- board text added: "HIGH"
- board text added: "INV"
- board text added: "IO0"
- board text added: "J26"
- board text added: "LOW"
- board text added: "NC"
- board text added: "PASS"
- board text added: "PHOTO_OUT_N"
- board text added: "PHOTO_OUT_P"
- board text added: "RX"
- board text added: "SEL"
- board text added: "SELP"
- board text added: "TX"
- board text removed: "PN1"
- board text removed: "POUTP/N"
- board text removed: "PP1"

Commit message: batch01 ready
Routing:
- net GNDA: track 259.3 -> 297.5 mm, vias 20 -> 178
- net 12V: track 171.5 -> 168.1 mm
- net GNDD: vias 27 -> 182
Other:
- board text added: "142x58mm"
- board text removed: "123.135x58mm"

Commit message: batch01 ready
Other:
- outline, holes or cut-outs redrawn
Changed lines of the file:
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@@
   (gr_circle (center 77.236 126.5) (end 76.9985 126.5) (layer "F.Paste") (width 0.475) (fill none))
   (gr_circle (center 76.236 75) (end 75.9985 75) (layer "F.Paste") (width 0.475) (fill none))
+  (gr_circle (center 203.86 129.84) (end 203.6225 129.84) (layer "F.Paste") (width 0.475) (fill none))
   (gr_circle (center 148.236 76) (end 147.9985 76) (layer "F.Paste") (width 0.475) (fill none))
+  (gr_circle (center 207.35 74.695) (end 207.1125 74.695) (layer "F.Paste") (width 0.475) (fill none))
   (gr_line (start 147.657227 111.5) (end 147.657227 92.5) (layer "F.SilkS") (width 0.1))
   (gr_arc (start 69.793791 87.266166) (mid 70.34204 87.588129) (end 70.761537 88.065895) (layer "F.SilkS") (width 0.1))
@@
   (gr_circle (center 76.236 75) (end 75.836 75) (layer "F.Mask") (width 0.475) (fill none))
   (gr_circle (center 148.236 128) (end 147.836 128) (layer "F.Mask") (width 0.475) (fill none))
+  (gr_circle (center 203.86 129.84) (end 203.46 129.84) (layer "F.Mask") (width 0.475) (fill none))
   (gr_circle (center 148.236 76) (end 147.836 76) (layer "F.Mask") (width 0.475) (fill none))
+  (gr_circle (center 207.35 74.695) (end 206.95 74.695) (layer "F.Mask") (width 0.475) (fill none))
   (gr_line (start 86.942944 74.501749) (end 87.296497 74.148195) (layer "Edge.Cuts") (width 0.1))
   (gr_line (start 111.357157 127.898251) (end 111.003604 127.544698) (layer "Edge.Cuts") (width 0.1))
@@
   (gr_line (start 124.357157 129.498251) (end 127.942944 129.498251) (layer "Edge.Cuts") (width 0.1))
   (gr_line (start 126.942944 74.501749) (end 127.296497 74.148195) (layer "Edge.Cuts") (width 0.1))
+  (gr_circle (center 203.86 129.84) (end 203.385 129.84) (layer "Edge.Cuts") (width 0.1) (fill none))
   (gr_line (start 124.357157 127.898251) (end 124.003604 127.544698) (layer "Edge.Cuts") (width 0.1))
   (gr_arc (start 114.296497 74.148195) (mid 114.841392 74.039809) (end 115.15005 74.50175) (layer "Edge.Cuts") (width 0.1))
+  (gr_circle (center 207.35 74.695) (end 206.875 74.695) (layer "Edge.Cuts") (width 0.1) (fill none))
   (gr_arc (start 129.15005 129.49825) (mid 128.841393 129.96019) (end 128.296497 129.851805) (layer "Edge.Cuts") (width 0.1))
   (gr_line (start 141.296497 76.455302) (end 140.942944 76.101749) (layer "Edge.Cuts") (width 0.1))
@@
     (effects (font (size 1 1) (thickness 0.15)) (justify mirror))
   )
-  (gr_text "HIGH" (at 188.06 87.07 270) (layer "B.SilkS")
+  (gr_text "HIGH" (at 188.06 87.07 90) (layer "B.SilkS")
     (effects (font (size 1 1) (thickness 0.15)) (justify mirror))
   )
@@
     (effects (font (size 0.508 0.508) (thickness 0.127)) (justify mirror))
   )
-  (gr_text "LOW" (at 188.03 77.96 270) (layer "B.SilkS")
-    (effects (font (size 1 1) (thickness 0.15)) (justify mirror))
-  )
+  (gr_text "LOW" (at 188.03 77.96 90) (layer "B.SilkS")
+    (effects (font (size 1 1) (thickness 0.15)) (justify mirror))
+  )
