File: kicad/NinjaLite/batch01/lcd/qLAMP-lcd.kicad_sch (KiCad schematic)
At the start: 22 parts, among them J1 Conn_01x04_Male, J2 Conn_01x04_Male, J3 Conn_01x04_Male, Q1 Q_NPN_BEC, Q2 Q_NPN_BEC, Q3 Q_NPN_BEC, SW1 TACTILE_4, SW2 TACTILE_4, SW3 TACTILE_4

Commit message: batch01 ready
Parts:
- R5, R7: value R -> 100k
Changed lines of the file:
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@@
       (effects (font (size 1.27 1.27)) (justify left))
     )
-    (property "Value" "R" (id 1) (at 79.248 70.4466 0)
+    (property "Value" "100k" (id 1) (at 79.248 70.4466 0)
       (effects (font (size 1.27 1.27)) (justify left))
     )
@@
       (effects (font (size 1.27 1.27)) (justify left))
     )
-    (property "Value" "R" (id 1) (at 85.598 70.4466 0)
+    (property "Value" "100k" (id 1) (at 85.598 70.4466 0)
       (effects (font (size 1.27 1.27)) (justify left))
     )
@@
     )
     (path "/548aa466-f8cf-4d32-a1b7-99b1cf19d7c2"
-      (reference "R5") (unit 1) (value "R") (footprint "Resistor_SMD:R_0603_1608Metric")
+      (reference "R5") (unit 1) (value "100k") (footprint "Resistor_SMD:R_0603_1608Metric")
     )
     (path "/bae238f1-3c6d-40d5-83da-e8948308d6d9"
@@
     )
     (path "/c9a613e5-ecd1-47c1-8de5-6361beee4d2c"
-      (reference "R7") (unit 1) (value "R") (footprint "Resistor_SMD:R_0603_1608Metric")
+      (reference "R7") (unit 1) (value "100k") (footprint "Resistor_SMD:R_0603_1608Metric")
     )
     (path "/717faf36-4f0d-408b-ae4a-a733881e3b95"
