File: kicad/NinjaLite/batch01/main_noADA/qLAMP-main.kicad_pcb (KiCad board)
At the start: 2 copper layers, 142 x 58 mm, 143 parts, among them J1 ALI_USB, J12 Conn_01x06_Male, J13 Conn_01x01_Male, J14 Conn_01x01_Male, J15 Conn_01x01_Male, J16 Conn_01x01_Male, J2 Barrel_Jack_Switch, J20 Conn_01x01_Male, J21 Conn_01x05_Male, J22 Conn_01x02_Male, J23 Conn_01x01_Male, J24 Conn_01x02_Male, J25 Conn_01x02_Male, J26 Conn_01x02_Male, J27 Conn_01x02_Male, J3 Conn_01x06_Male, Q1 Q_NMOS_GSD, Q3 Q_NMOS_GSD, Q5 Q_NMOS_GSD, U1 ADA2200ARUZ, U10 TLC5929, U11 IP2721, U12 TPS63710DRRR, U13 MCP1755T-3302E_DC, U14 MCP1755T-3302E_OT, U15 CJT1117-3.3, U16 CJT1117-5.0, U17 LITE_LCD, U19 CD74HC4067M96, U2 ADS1219IPWR, U3 COM1305-0.032768-EXT-T-TR, U4 LMP7717MF_NOPB, U5 ESP32-WROOM-32, U7 SN74LVC1GU04DCKR, U8 TS12A12511DCNR, U9 SN74LV4051A

Commit message: sync
Parts:
- removed C1, C2: 4.7uF, Capacitor_SMD:C_0805_2012Metric
- removed C7: 0.1uF, Capacitor_SMD:C_0603_1608Metric
- removed J12: Conn_01x06_Male, Connector_PinSocket_1.27mm:PinSocket_1x06_P1.27mm_Vertical
- removed J14, J15: Conn_01x01_Male, Connector_PinSocket_1.27mm:PinSocket_1x01_P1.27mm_Vertical
- removed J20: Conn_01x01_Male, Connector_PinHeader_1.27mm:PinHeader_1x01_P1.27mm_Vertical
- removed J21: Conn_01x05_Male, Connector_PinSocket_1.27mm:PinSocket_1x05_P1.27mm_Vertical
- removed J22: Conn_01x02_Male, Connector_PinHeader_1.27mm:PinHeader_1x02_P1.27mm_Vertical
- removed JP4, JP5, JP8: Jumper_3_Open, Jumper:SolderJumper-3_P2.0mm_Open_TrianglePad1.0x1.5mm
- removed R10, R11, R14: 10k, Resistor_SMD:R_0603_1608Metric
- removed U3: COM1305-0.032768-EXT-T-TR, Ninja-qPCR:ASDK-32.768KHZ-LRT
- removed U7: SN74LVC1GU04DCKR, Ninja-qPCR:SN74LVC1GU04DBVR
- U1: value ADA2200ARUZ -> MCP3426; footprint Ninja-qPCR:ADA2200ARUZ -> Package_SO:SOIC-8_3.9x4.9mm_P1.27mm
- moved U1 0.68 mm to (101.8, 101.8), turned to 180 degrees
Connections:
- C5 pad 1: /Photo/PHOTO_OUT_N -> GNDA
- C5 pad 2: /Photo/PHOTO_OUT_P -> /Photo/LPF_OUT
- U1 pad 1: CLKIN -> THERM_MUX_OUT
- U1 pad 2: unconnected-(U1-Pad2) -> GNDA
- U1 pad 3: unconnected-(U1-Pad3) -> 3V3D
- U1 pad 4: /Photo/ADA4 -> I2C_SDA
- U1 pad 5: GNDD -> I2C_SCL
- U1 pad 6: /Photo/LPF_OUT -> GNDD
- U1 pad 7: GNDA -> /Photo/LPF_OUT
- U1 pad 8: /Photo/ADA8 -> GNDA
- U10 pad 21: /PhotoLED/LED_BLANK -> LED_BLANK
- U10 pad 22: LED_SPI_MISO -> unconnected-(U10-Pad22)
- U2 pad 6: /Photo/PHOTO_OUT_P -> /Photo/LPF_OUT
- U2 pad 7: /Photo/PHOTO_OUT_N -> GNDA
- U5 pad 23: LED_SPI_MISO -> LED_BLANK
Routing:
- net PD_REF_PWM: track 97.8 -> 0.00 mm, vias 3 -> 0
- net LED_BLANK: track 0.00 -> 95.2 mm, vias 0 -> 2
- net (no net): track 0.00 -> 95.1 mm, vias 0 -> 4
- net LED_SPI_MISO: track 60.6 -> 0.00 mm, vias 2 -> 0
- net /PhotoLED/LED_BLANK: track 37.7 -> 0.00 mm, vias 1 -> 0
- net /Photo/PHOTO_OUT_P: track 34.8 -> 0.00 mm, vias 2 -> 0
- net /Photo/LPF_OUT: track 16.6 -> 47.7 mm, vias 0 -> 1
- net /Photo/PHOTO_OUT_N: track 30.7 -> 0.00 mm, vias 1 -> 0
- net /Photo/PP1: track 25.7 -> 0.00 mm, vias 2 -> 0
- net /Photo/PN1: track 23.8 -> 0.00 mm, vias 3 -> 0
- net /Photo/PN2: track 23.4 -> 0.00 mm, vias 1 -> 0
- net I2C_SCL: track 152.6 -> 173.2 mm
- net 3V3D: track 322.5 -> 305.7 mm, vias 17 -> 19
- net GNDD: track 569.7 -> 553.8 mm
- net THERM_MUX_OUT: track 125.1 -> 140.7 mm, vias 6 -> 7
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Other:
- board text added: "batch01/main_noADA_newADC"
- board text removed: "batch01/main"
