File: kicad/NinjaLite/batch01/photo-single/photo-single.kicad_pcb (KiCad board)
At the start: 2 copper layers, 123.1 x 58 mm, 31 parts, among them J1 Conn_01x60_Male

Commit message: sync
Changed lines of the file:
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@@
   (gr_arc (start 103.545497 80.855302) (mid 103.437111 80.310407) (end 103.89905 80.00175) (layer "Edge.Cuts") (width 0.1))
   (gr_line (start 146.91405 72.501749) (end 146.91405 74.101749) (layer "Edge.Cuts") (width 0.1))
-  (gr_arc (start 159.060497 72.148195) (mid 159.605392 72.039809) (end 159.91405 72.50175) (layer "Edge.Cuts") (width 0.1))
+  (gr_arc (start 159.060497 72.148195) (mid 159.605393 72.039809) (end 159.91405 72.50175) (layer "Edge.Cuts") (width 0.1))
   (gr_line (start 207.399 71) (end 85.264 71) (layer "Edge.Cuts") (width 0.1))
   (gr_line (start 156.121157 72.501749) (end 158.706944 72.501749) (layer "Edge.Cuts") (width 0.1))
@@
   (gr_line (start 141.767604 72.148195) (end 142.121157 72.501749) (layer "Edge.Cuts") (width 0.1))
   (gr_line (start 103.89905 84.894642) (end 103.89905 81.208855) (layer "Edge.Cuts") (width 0.1))
-  (gr_arc (start 132.060497 72.148195) (mid 132.605392 72.039809) (end 132.91405 72.50175) (layer "Edge.Cuts") (width 0.1))
+  (gr_arc (start 132.060497 72.148195) (mid 132.605393 72.039809) (end 132.91405 72.50175) (layer "Edge.Cuts") (width 0.1))
   (gr_line (start 158.706944 72.501749) (end 159.060497 72.148195) (layer "Edge.Cuts") (width 0.1))
   (gr_line (start 146.545497 85.248195) (end 146.89905 84.894642) (layer "Edge.Cuts") (width 0.1))
   (gr_line (start 155.767604 72.148195) (end 156.121157 72.501749) (layer "Edge.Cuts") (width 0.1))
-  (gr_arc (start 105.060497 72.148195) (mid 105.605392 72.039809) (end 105.91405 72.50175) (layer "Edge.Cuts") (width 0.1))
+  (gr_arc (start 105.060497 72.148195) (mid 105.605393 72.039809) (end 105.91405 72.50175) (layer "Edge.Cuts") (width 0.1))
   (gr_arc (start 141.767604 74.455302) (mid 141.222709 74.563689) (end 140.91405 74.10175) (layer "Edge.Cuts") (width 0.1))
   (gr_line (start 100.91405 74.101749) (end 100.91405 72.501749) (layer "Edge.Cuts") (width 0.1))
@@
   (gr_line (start 103.545497 85.248195) (end 103.89905 84.894642) (layer "Edge.Cuts") (width 0.1))
   (gr_line (start 113.89905 84.894642) (end 114.252604 85.248195) (layer "Edge.Cuts") (width 0.1))
-  (gr_arc (start 146.060497 72.148195) (mid 146.605392 72.039809) (end 146.91405 72.50175) (layer "Edge.Cuts") (width 0.1))
+  (gr_arc (start 146.060497 72.148195) (mid 146.605393 72.039809) (end 146.91405 72.50175) (layer "Edge.Cuts") (width 0.1))
   (gr_line (start 145.706944 74.101749) (end 142.121157 74.101749) (layer "Edge.Cuts") (width 0.1))
   (gr_line (start 156.89905 86.101749) (end 146.89905 86.101749) (layer "Edge.Cuts") (width 0.1))
@@
   (gr_line (start 127.91405 74.101749) (end 127.91405 72.501749) (layer "Edge.Cuts") (width 0.1))
   (gr_arc (start 127.91405 72.501749) (mid 128.222708 72.039809) (end 128.767603 72.148196) (layer "Edge.Cuts") (width 0.1))
-  (gr_arc (start 119.060497 72.148195) (mid 119.605392 72.039809) (end 119.91405 72.50175) (layer "Edge.Cuts") (width 0.1))
+  (gr_arc (start 119.060497 72.148195) (mid 119.605393 72.039809) (end 119.91405 72.50175) (layer "Edge.Cuts") (width 0.1))
   (gr_line (start 129.121157 74.101749) (end 128.767604 74.455302) (layer "Edge.Cuts") (width 0.1))
   (gr_arc (start 156.89905 80.001749) (mid 157.36099 80.310407) (end 157.252603 80.855302) (layer "Edge.Cuts") (width 0.1))
