File: kicad/NinjaLite/batch02/main/qLAMP-main.kicad_pcb (KiCad board)
At the start: 2 copper layers, 142 x 58 mm, 143 parts, among them J1 ALI_USB, J12 Conn_01x06_Male, J13 Conn_01x01_Male, J14 Conn_01x01_Male, J15 Conn_01x01_Male, J16 Conn_01x01_Male, J2 Barrel_Jack_Switch, J20 Conn_01x01_Male, J21 Conn_01x05_Male, J22 Conn_01x02_Male, J23 Conn_01x01_Male, J24 Conn_01x02_Male, J25 Conn_01x02_Male, J26 Conn_01x02_Male, J27 Conn_01x02_Male, J3 Conn_01x06_Male, Q1 Q_NMOS_GSD, Q3 Q_NMOS_GSD, Q5 Q_NMOS_GSD, U1 ADA2200ARUZ, U10 TLC5929, U11 IP2721, U12 TPS63710DRRR, U13 MCP1755T-3302E_DC, U14 MCP1755T-3302E_OT, U15 CJT1117-3.3, U16 CJT1117-5.0, U17 LITE_LCD, U19 CD74HC4067M96, U2 ADS1219IPWR, U3 COM1305-0.032768-EXT-T-TR, U4 LMP7717MF_NOPB, U5 ESP32-WROOM-32, U7 SN74LVC1GU04DCKR, U8 TS12A12511DCNR, U9 SN74LV4051A

Commit message: sync
Parts:
- removed C1, C2: 4.7uF, Capacitor_SMD:C_0805_2012Metric
- removed C7: 0.1uF, Capacitor_SMD:C_0603_1608Metric
- removed J12: Conn_01x06_Male, Connector_PinSocket_1.27mm:PinSocket_1x06_P1.27mm_Vertical
- removed J14, J15: Conn_01x01_Male, Connector_PinSocket_1.27mm:PinSocket_1x01_P1.27mm_Vertical
- removed J20: Conn_01x01_Male, Connector_PinHeader_1.27mm:PinHeader_1x01_P1.27mm_Vertical
- removed J21: Conn_01x05_Male, Connector_PinSocket_1.27mm:PinSocket_1x05_P1.27mm_Vertical
- removed J22: Conn_01x02_Male, Connector_PinHeader_1.27mm:PinHeader_1x02_P1.27mm_Vertical
- removed JP4, JP5, JP8: Jumper_3_Open, Jumper:SolderJumper-3_P2.0mm_Open_TrianglePad1.0x1.5mm
- removed R10, R11, R14: 10k, Resistor_SMD:R_0603_1608Metric
- removed U3: COM1305-0.032768-EXT-T-TR, Ninja-qPCR:ASDK-32.768KHZ-LRT
- removed U7: SN74LVC1GU04DCKR, Ninja-qPCR:SN74LVC1GU04DBVR
- U1: value ADA2200ARUZ -> MCP3426; footprint Ninja-qPCR:ADA2200ARUZ -> Package_SO:SOIC-8_3.9x4.9mm_P1.27mm
- moved C13 1.88 mm to (196.0, 81.8)
- moved Q1 1.85 mm to (195.8, 84.6)
- moved U1 0.68 mm to (101.8, 101.8), turned to 180 degrees
Connections:
- C5 pad 1: /Photo/PHOTO_OUT_N -> GNDA
- C5 pad 2: /Photo/PHOTO_OUT_P -> /Photo/LPF_OUT
- U1 pad 1: CLKIN -> THERM_MUX_OUT
- U1 pad 2: unconnected-(U1-Pad2) -> GNDA
- U1 pad 3: unconnected-(U1-Pad3) -> 3V3D
- U1 pad 4: /Photo/ADA4 -> I2C_SDA
- U1 pad 5: GNDD -> I2C_SCL
- U1 pad 6: /Photo/LPF_OUT -> GNDD
- U1 pad 7: GNDA -> /Photo/LPF_OUT
- U1 pad 8: /Photo/ADA8 -> GNDA
- U10 pad 21: /PhotoLED/LED_BLANK -> LED_BLANK
- U10 pad 22: LED_SPI_MISO -> unconnected-(U10-Pad22)
- U2 pad 6: /Photo/PHOTO_OUT_P -> /Photo/LPF_OUT
- U2 pad 7: /Photo/PHOTO_OUT_N -> GNDA
- U5 pad 23: LED_SPI_MISO -> LED_BLANK
Routing:
- net PD_REF_PWM: track 97.8 -> 0.00 mm, vias 3 -> 0
- net LED_BLANK: track 0.00 -> 95.2 mm, vias 0 -> 2
- net (no net): track 0.00 -> 95.1 mm, vias 0 -> 4
- net LED_SPI_MISO: track 60.6 -> 0.00 mm, vias 2 -> 0
- net /PhotoLED/LED_BLANK: track 37.7 -> 0.00 mm, vias 1 -> 0
- net /Photo/PHOTO_OUT_P: track 34.8 -> 0.00 mm, vias 2 -> 0
- net /Photo/LPF_OUT: track 16.6 -> 47.7 mm, vias 0 -> 1
- net /Photo/PHOTO_OUT_N: track 30.7 -> 0.00 mm, vias 1 -> 0
- net /Photo/PP1: track 25.7 -> 0.00 mm, vias 2 -> 0
- net /Photo/PN1: track 23.8 -> 0.00 mm, vias 3 -> 0
- net /Photo/PN2: track 23.4 -> 0.00 mm, vias 1 -> 0
- net I2C_SCL: track 152.6 -> 173.2 mm
- net 3V3D: track 322.5 -> 305.7 mm, vias 17 -> 19
- net THERM_MUX_OUT: track 125.1 -> 140.7 mm, vias 6 -> 7
- net GNDD: track 569.7 -> 557.9 mm
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Other:
- outline, holes or cut-outs redrawn
- board text added: "batch01/main_noADA_newADC"
- board text removed: "batch01/main"

Commit message: fix
Parts:
- removed C30: 100pF, Capacitor_SMD:C_0603_1608Metric
- removed U13: MCP1755T-3302E_DC, Package_TO_SOT_SMD:SOT-223-6
- removed U15: CJT1117-3.3, Package_TO_SOT_SMD:SOT-223
- removed U16: CJT1117-5.0, Package_TO_SOT_SMD:SOT-223
- added C1: 0.1uF, Capacitor_SMD:C_0603_1608Metric, F.Cu at (191.7, 58.1)
- added U3: BD433M5FP-CE2, Ninja-qPCR:REG_TO252-3, F.Cu at (178.1, 61.1)
- added U6: BA178M05FP-E2, Ninja-qPCR:REG_TO252-3, F.Cu at (163.8, 61.1)
- C18: value 330pF -> DNP
- C6: value DNP(<1pF) -> 5pF
- C8: value 0.1uF -> DNP
- R13: value 10M -> 20M
- R2: value 0 -> 3.3k
- U1: value MCP3426 -> NAU7802; footprint Package_SO:SOIC-8_3.9x4.9mm_P1.27mm -> Package_DIP:DIP-16_W7.62mm
- U14: value MCP1755T-3302E_OT -> TCR3DF33,LM(CT
Connections:
- C17 pad 1: 12V -> 20V
- C22 pad 1: 12V -> Net-(C22-Pad1)
- C23 pad 1: 12V -> 20V
- C24 pad 1: 12V -> Net-(C22-Pad1)
- C25 pad 1: 12V -> 20V
- C26 pad 1: 12V -> Net-(C22-Pad1)
- C27 pad 1: 12V -> 20V
- HLID1 pad 1: 12V -> 20V
- HWELL1 pad 1: 12V -> 20V
- J2 pad 1: 12V -> 20V
- Q1 pad 2: 12V -> 20V
- R16 pad 2: 12V -> 20V
- R19 pad 1: 12V -> 20V
- U1 pad 1: THERM_MUX_OUT -> 3V3A
- U1 pad 2: GNDA -> DIVIDED
- U1 pad 3: 3V3D -> THERM_MUX_OUT
- U1 pad 4: I2C_SDA -> DIVIDED
- U1 pad 5: I2C_SCL -> /Photo/LPF_OUT
- U1 pad 6: GNDD -> Net-(C1-Pad1)
- U1 pad 7: /Photo/LPF_OUT -> GNDA
- U11 pad 16: 12V -> 20V
- U14 pad 1: 12V -> Net-(C22-Pad1)
- U14 pad 3: 12V -> Net-(C22-Pad1)
- U14 pad 4: /Power/PWRGD -> unconnected-(U14-Pad4)
- U17 pad 11: LED_G -> unconnected-(U17-Pad11)
- U17 pad 12: LED_B -> unconnected-(U17-Pad12)
- U19 pad 15: 3V3D -> -1V
- U5 pad 10: LED_G -> /LID_HEATER
- U5 pad 11: LED_B -> /WELL_HEATER
- U5 pad 6: /WELL_HEATER -> unconnected-(U5-Pad6)
- U5 pad 7: /LID_HEATER -> unconnected-(U5-Pad7)
Routing:
- net GNDD: track 557.9 -> 731.1 mm, vias 182 -> 186
- net I2C_SCL: track 173.2 -> 0.00 mm, vias 4 -> 0
- net 20V: track 0.00 -> 167.4 mm, vias 0 -> 2
- net 12V: track 167.4 -> 0.00 mm, vias 2 -> 0
- net GNDA: track 289.4 -> 339.4 mm, vias 190 -> 192
- net /Photo/LPF_OUT: track 47.7 -> 0.00 mm, vias 1 -> 0
- net LED_B: track 41.8 -> 0.00 mm, vias 2 -> 0
- net /WELL_HEATER: track 13.4 -> 55.2 mm, vias 0 -> 2
- net LED_G: track 40.7 -> 0.00 mm, vias 2 -> 0
- net /LID_HEATER: track 22.7 -> 63.3 mm, vias 0 -> 2
- net unconnected-(U14-Pad4): track 0.00 -> 10.7 mm, vias 0 -> 2
- net /Power/PWRGD: track 10.7 -> 0.00 mm, vias 2 -> 0
- net Net-(C18-Pad1): track 2.34 -> 0.00 mm, vias 1 -> 0
- added copper zone on F.Cu, net 20V
- removed copper zone on F.Cu, net 12V

Commit message: sync
Parts:
- moved U1 14.4 mm to (115.6, 97.8), turned to -90 degrees
Routing:
- net Net-(C18-Pad1): track 0.00 -> 2.34 mm, vias 0 -> 1
- net GNDA: track 339.4 -> 337.1 mm, vias 192 -> 191
Other:
- board text added: "batch02/main"
- board text removed: "batch01/main_noADA_newADC"
Changed lines of the file:
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@@
   )
   (footprint "Package_DIP:DIP-16_W7.62mm" (layer "F.Cu")
-    (at 101.76 101.79 180)
+    (at 115.555 97.78 -90)
     (descr "16-lead though-hole mounted DIP package, row spacing 7.62 mm (300 mils)")
     (tags "THT DIP DIL PDIP 2.54mm 7.62mm 300mil")
@@
     (property "Sheetname" "Photo")
     (attr through_hole)
-    (fp_text reference "U1" (at 3.81 -2.33 180) (layer "F.SilkS")
+    (fp_text reference "U1" (at 3.81 -2.33 90) (layer "F.SilkS")
       (effects (font (size 1 1) (thickness 0.15)))
     )
-    (fp_text value "NAU7802" (at 3.81 20.11 180) (layer "F.Fab")
+    (fp_text value "NAU7802" (at 3.81 20.11 90) (layer "F.Fab")
       (effects (font (size 1 1) (thickness 0.15)))
     )
-    (fp_text user "${REFERENCE}" (at 3.81 8.89 180) (layer "F.Fab")
+    (fp_text user "${REFERENCE}" (at 3.81 8.89 90) (layer "F.Fab")
       (effects (font (size 1 1) (thickness 0.15)))
     )
@@
     (fp_line (start 1.635 -1.27) (end 6.985 -1.27) (layer "F.Fab") (width 0.1))
     (fp_line (start 0.635 19.05) (end 0.635 -0.27) (layer "F.Fab") (width 0.1))
-    (pad "1" thru_hole rect (at 0 0 180) (size 1.6 1.6) (drill 0.8) (layers *.Cu *.Mask)
+    (pad "1" thru_hole rect (at 0 0 270) (size 1.6 1.6) (drill 0.8) (layers *.Cu *.Mask)
       (net 4 "3V3A") (pinfunction "REFP") (pintype "input"))
-    (pad "2" thru_hole oval (at 0 2.54 180) (size 1.6 1.6) (drill 0.8) (layers *.Cu *.Mask)
+    (pad "2" thru_hole oval (at 0 2.54 270) (size 1.6 1.6) (drill 0.8) (layers *.Cu *.Mask)
       (net 134 "DIVIDED") (pinfunction "VIN1N") (pintype "input"))
-    (pad "3" thru_hole oval (at 0 5.08 180) (size 1.6 1.6) (drill 0.8) (layers *.Cu *.Mask)
+    (pad "3" thru_hole oval (at 0 5.08 270) (size 1.6 1.6) (drill 0.8) (layers *.Cu *.Mask)
       (net 23 "THERM_MUX_OUT") (pinfunction "VIN1P") (pintype "input"))
-    (pad "4" thru_hole oval (at 0 7.62 180) (size 1.6 1.6) (drill 0.8) (layers *.Cu *.Mask)
+    (pad "4" thru_hole oval (at 0 7.62 270) (size 1.6 1.6) (drill 0.8) (layers *.Cu *.Mask)
       (net 134 "DIVIDED") (pinfunction "VIN2N") (pintype "input"))
-    (pad "5" thru_hole oval (at 0 10.16 180) (size 1.6 1.6) (drill 0.8) (layers *.Cu *.Mask)
+    (pad "5" thru_hole oval (at 0 10.16 270) (size 1.6 1.6) (drill 0.8) (layers *.Cu *.Mask)
       (net 58 "/Photo/LPF_OUT") (pinfunction "VIN2P") (pintype "input"))
-    (pad "6" thru_hole oval (at 0 12.7 180) (size 1.6 1.6) (drill 0.8) (layers *.Cu *.Mask)
+    (pad "6" thru_hole oval (at 0 12.7 270) (size 1.6 1.6) (drill 0.8) (layers *.Cu *.Mask)
       (net 142 "Net-(C1-Pad1)") (pinfunction "VBG") (pintype "input"))
-    (pad "7" thru_hole oval (at 0 15.24 180) (size 1.6 1.6) (drill 0.8) (layers *.Cu *.Mask)
+    (pad "7" thru_hole oval (at 0 15.24 270) (size 1.6 1.6) (drill 0.8) (layers *.Cu *.Mask)
       (net 2 "GNDA") (pinfunction "REFN") (pintype "input"))
-    (pad "8" thru_hole oval (at 0 17.78 180) (size 1.6 1.6) (drill 0.8) (layers *.Cu *.Mask)
+    (pad "8" thru_hole oval (at 0 17.78 270) (size 1.6 1.6) (drill 0.8) (layers *.Cu *.Mask)
       (net 2 "GNDA") (pinfunction "AVSS") (pintype "input"))
-    (pad "9" thru_hole oval (at 7.62 17.78 180) (size 1.6 1.6) (drill 0.8) (layers *.Cu *.Mask)
+    (pad "9" thru_hole oval (at 7.62 17.78 270) (size 1.6 1.6) (drill 0.8) (layers *.Cu *.Mask)
       (net 43 "GNDD") (pinfunction "DVSS") (pintype "input"))
-    (pad "10" thru_hole oval (at 7.62 15.24 180) (size 1.6 1.6) (drill 0.8) (layers *.Cu *.Mask)
+    (pad "10" thru_hole oval (at 7.62 15.24 270) (size 1.6 1.6) (drill 0.8) (layers *.Cu *.Mask)
       (net 143 "unconnected-(U1-Pad10)") (pinfunction "XIN") (pintype "input"))
-    (pad "11" thru_hole oval (at 7.62 12.7 180) (size 1.6 1.6) (drill 0.8) (layers *.Cu *.Mask)
+    (pad "11" thru_hole oval (at 7.62 12.7 270) (size 1.6 1.6) (drill 0.8) (layers *.Cu *.Mask)
       (net 144 "unconnected-(U1-Pad11)") (pinfunction "XOUT") (pintype "input"))
-    (pad "12" thru_hole oval (at 7.62 10.16 180) (size 1.6 1.6) (drill 0.8) (layers *.Cu *.Mask)
+    (pad "12" thru_hole oval (at 7.62 10.16 270) (size 1.6 1.6) (drill 0.8) (layers *.Cu *.Mask)
       (net 145 "unconnected-(U1-Pad12)") (pinfunction "DRDY") (pintype "input"))
-    (pad "13" thru_hole oval (at 7.62 7.62 180) (size 1.6 1.6) (drill 0.8) (layers *.Cu *.Mask)
+    (pad "13" thru_hole oval (at 7.62 7.62 270) (size 1.6 1.6) (drill 0.8) (layers *.Cu *.Mask)
       (net 146 "unconnected-(U1-Pad13)") (pinfunction "SCLK") (pintype "input"))
-    (pad "14" thru_hole oval (at 7.62 5.08 180) (size 1.6 1.6) (drill 0.8) (layers *.Cu *.Mask)
+    (pad "14" thru_hole oval (at 7.62 5.08 270) (size 1.6 1.6) (drill 0.8) (layers *.Cu *.Mask)
       (net 147 "unconnected-(U1-Pad14)") (pinfunction "SDIO") (pintype "input"))
-    (pad "15" thru_hole oval (at 7.62 2.54 180) (size 1.6 1.6) (drill 0.8) (layers *.Cu *.Mask)
+    (pad "15" thru_hole oval (at 7.62 2.54 270) (size 1.6 1.6) (drill 0.8) (layers *.Cu *.Mask)
       (net 3 "3V3D") (pinfunction "DVDD") (pintype "input"))
-    (pad "16" thru_hole oval (at 7.62 0 180) (size 1.6 1.6) (drill 0.8) (layers *.Cu *.Mask)
+    (pad "16" thru_hole oval (at 7.62 0 270) (size 1.6 1.6) (drill 0.8) (layers *.Cu *.Mask)
       (net 4 "3V3A") (pinfunction "AVDD") (pintype "input"))
     (model "${KICAD6_3DMODEL_DIR}/Package_DIP.3dshapes/DIP-16_W7.62mm.wrl"
@@
     (effects (font (size 0.508 0.508) (thickness 0.127)) (justify mirror))
   )
-  (gr_text "batch01/main_noADA_newADC\n" (at 121.92 125.420018) (layer "F.SilkS")
+  (gr_text "batch02/main" (at 121.92 125.420018) (layer "F.SilkS")
     (effects (font (size 1.2 1.2) (thickness 0.254)))
   )
@@
   (segment (start 114.54 103.61) (end 114.726 103.796) (width 0.21082) (layer "F.Cu") (net 2))
   (segment (start 89.726 96.26) (end 91.126 94.86) (width 0.21082) (layer "F.Cu") (net 2))
-  (segment (start 92.776006 99.135012) (end 92.841005 99.135012) (width 0.21082) (layer "F.Cu") (net 2))
   (segment (start 94.764135 101.844135) (end 94.764135 97.434135) (width 0.21082) (layer "F.Cu") (net 2))
   (segment (start 113.426 103.79418) (end 113.426 104.79) (width 0.21082) (layer "F.Cu") (net 2))
@@
   (segment (start 115.740002 100.41001) (end 115.516473 100.633539) (width 0.21082) (layer "F.Cu") (net 2))
   (segment (start 145.156 94.003277) (end 145.157211 94.002066) (width 0.762) (layer "F.Cu") (net 2))
-  (segment (start 92.841005 99.135012) (end 94.146005 100.440012) (width 0.21082) (layer "F.Cu") (net 2))
   (segment (start 109.306 107.2) (end 108.799004 107.2) (width 0.21082) (layer "F.Cu") (net 2))
   (segment (start 113.61 96.63) (end 113.55913 96.68087) (width 0.21082) (layer "F.Cu") (net 2))
@@
   (via (at 72.92 82.17) (size 0.8) (drill 0.4) (layers "F.Cu" "B.Cu") (free) (net 2))
   (via (at 139.2 109.86) (size 0.8) (drill 0.4) (layers "F.Cu" "B.Cu") (free) (net 2))
-  (via (at 92.776006 99.135012) (size 0.8) (drill 0.4) (layers "F.Cu" "B.Cu") (net 2))
   (via (at 84.47 79.07) (size 0.8) (drill 0.4) (layers "F.Cu" "B.Cu") (free) (net 2))
   (via (at 147.45 89.59) (size 0.8) (drill 0.4) (layers "F.Cu" "B.Cu") (free) (net 2))
@@
   (segment (start 92.854119 109.018119) (end 92.866 109.03) (width 0.21082) (layer "B.Cu") (net 2))
   (segment (start 110.970009 102.299999) (end 109.550022 102.299999) (width 0.21082) (layer "B.Cu") (net 2))
-  (segment (start 92.616 99.5) (end 92.616 99.295018) (width 0.21082) (layer "B.Cu") (net 2))
   (segment (start 115.627661 107.908339) (end 111.09057 107.908339) (width 0.21082) (layer "B.Cu") (net 2))
   (segment (start 149.12 96.45) (end 152.4 96.45) (width 0.21082) (layer "B.Cu") (net 2))
@@
   (segment (start 90.616 98.4) (end 91.097874 97.918126) (width 0.21082) (layer "B.Cu") (net 2))
   (segment (start 159.646956 93.119052) (end 161.580948 93.119052) (width 0.21082) (layer "B.Cu") (net 2))
-  (segment (start 92.616 99.295018) (end 92.776006 99.135012) (width 0.21082) (layer "B.Cu") (net 2))
   (segment (start 87.716 105.54375) (end 87.997877 105.261873) (width 0.21082) (layer "B.Cu") (net 2))
   (segment (start 113.31001 101.000001) (end 112.270007 101.000001) (width 0.21082) (layer "B.Cu") (net 2))
@@
   (segment (start 89.651 104.275) (end 90.508 104.275) (width 0.21082) (layer "F.Cu") (net 54))
   (via (at 88.52379 103.777677) (size 0.8) (drill 0.4) (layers "F.Cu" "B.Cu") (net 54))
+  (segment (start 92.776006 99.135012) (end 92.841005 99.135012) (width 0.21082) (layer "F.Cu") (net 55))
+  (segment (start 92.841005 99.135012) (end 94.146005 100.440012) (width 0.21082) (layer "F.Cu") (net 55))
+  (via (at 92.776006 99.135012) (size 0.8) (drill 0.4) (layers "F.Cu" "B.Cu") (net 55))
+  (segment (start 92.616 99.5) (end 92.616 99.295018) (width 0.21082) (layer "B.Cu") (net 55))
+  (segment (start 92.616 99.295018) (end 92.776006 99.135012) (width 0.21082) (layer "B.Cu") (net 55))
   (segment (start 94.236 106.419992) (end 94.235998 106.419994) (width 0.21082) (layer "F.Cu") (net 56))
   (segment (start 93.897873 105.611873) (end 94.235998 105.949998) (width 0.21082) (layer "B.Cu") (net 56))

Commit message: sync
Parts:
- removed C16: 1uF, Capacitor_SMD:C_0603_1608Metric
- removed C19: 10uF, Capacitor_SMD:C_0805_2012Metric
- removed C20, C21: 22uF, Capacitor_SMD:C_1210_3225Metric
- removed R15: 150k, Resistor_SMD:R_0603_1608Metric
- removed U12: TPS63710DRRR, Ninja-qPCR:TPS63710DRRR
- added C2: 0.1uF, Capacitor_SMD:C_0603_1608Metric, F.Cu at (125.4, 63.9)
- added C7: 22uF, Capacitor_SMD:C_1210_3225Metric, F.Cu at (134.7, 58.3)
- added D1: D_Schottky, Ninja-qPCR:MSS1P3L-M3&slash_89A, F.Cu at (134.0, 61.8)
- added JP2: Jumper_2_Bridged, Jumper:SolderJumper-2_P1.3mm_Open_TrianglePad1.0x1.5mm, B.Cu at (197.9, 129.2)
- added R10: 47k_HP, Resistor_SMD:R_0603_1608Metric, F.Cu at (144.4, 57.4)
- added R11: 47k_HP, Resistor_SMD:R_0603_1608Metric, F.Cu at (148.4, 57.4)
- added U7: AZ34063U, Package_SO:SOP-8_3.9x4.9mm_P1.27mm, F.Cu at (127.7, 59.4)
- C14: value 1uF -> 22uF; footprint Capacitor_SMD:C_0603_1608Metric -> Capacitor_SMD:C_1210_3225Metric
- J3: value Conn_01x06_Male -> Conn_01x07_Male; footprint Connector_PinHeader_2.54mm:PinHeader_1x06_P2.54mm_Vertical -> Connector_PinSocket_2.54mm:PinSocket_1x07_P2.54mm_Horizontal
- L1: value 2.2uH -> 68uH; footprint Capacitor_SMD:C_0805_2012Metric -> Inductor_SMD:L_Taiyo-Yuden_NR-60xx
- R5: value 39k -> 0.24
Connections:
- net LED_R renamed LED
- C14 pad 1: Net-(C14-Pad1) -> DIVIDED
- C14 pad 2: GNDD -> GNDA
- J3 pad 1: GNDD -> TACT2
- J3 pad 2: TACT2 -> GNDD
- J3 pad 3: /TXD -> unconnected-(J3-Pad3)
- J3 pad 4: /RXD -> Net-(J3-Pad4)
- J3 pad 5: GNDD -> /RXD
- J3 pad 6: unconnected-(J3-Pad6) -> /TXD
- L1 pad 2: -1V -> GNDD
- R5 pad 2: Net-(R15-Pad1) -> 3V3D
- U1 pad 12: unconnected-(U1-Pad12) -> NAU_DRDY
- U1 pad 13: unconnected-(U1-Pad13) -> I2C_SCL
- U1 pad 14: unconnected-(U1-Pad14) -> I2C_SDA
- U5 pad 27: unconnected-(U5-Pad27) -> NAU_DRDY
Routing:
- net GNDD: track 731.1 -> 1717.9 mm, vias 186 -> 240
- net GNDA: track 337.1 -> 27.4 mm, vias 191 -> 170
- net 3V3D: track 305.7 -> 0.00 mm, vias 19 -> 0
- net I2C_SDA: track 158.7 -> 0.00 mm, vias 5 -> 0
- net THERM_MUX_OUT: track 140.7 -> 0.00 mm, vias 7 -> 0
- net 3V3A: track 73.9 -> 0.00 mm, vias 2 -> 0
- net unconnected-(U17-Pad12): track 0.00 -> 41.8 mm, vias 0 -> 2
- net /WELL_HEATER: track 55.2 -> 13.4 mm, vias 2 -> 0
- net unconnected-(U17-Pad11): track 0.00 -> 40.7 mm, vias 0 -> 2
- net /LID_HEATER: track 63.3 -> 22.7 mm, vias 2 -> 0
- net DIVIDED: track 0.00 -> 9.78 mm
- net Net-(R15-Pad1): track 6.87 -> 0.00 mm
- net -1V: track 76.2 -> 81.4 mm
- net (no net): track 95.1 -> 99.1 mm
- net Net-(L1-Pad1): track 3.32 -> 0.00 mm
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