File: kicad/NinjaLite/batch02/main/filePower.kicad_sch (KiCad schematic)
At the start: 40 parts, among them J1 ALI_USB, J2 Barrel_Jack_Switch, Q1 Q_NMOS_GSD, U11 IP2721, U12 TPS63710DRRR, U13 MCP1755T-3302E_DC, U14 MCP1755T-3302E_OT, U15 CJT1117-3.3, U16 CJT1117-5.0

Commit message: sync
Parts:
- removed C30: 100pF, Capacitor_SMD:C_0603_1608Metric, symbol Device:C
- removed U13: MCP1755T-3302E_DC, Package_TO_SOT_SMD:SOT-223-6, symbol Ninja-qPCR:MCP1755T-3302E_DC
- U14: value MCP1755T-3302E_OT -> TCR3DF33,LM(CT
Connections:
- net 12V renamed 20V
- net 20V: no longer C22.1, C24.1, C26.1, U14.1 (VIN), U14.3 (SHDN)
- net PWRGD: no longer names the net of U14.4 (PWRGD)
- new net: C22.1, C24.1, C26.1, U14.1 (VIN), U14.3 (SHDN)
- no-connect marks 1 -> 2
Other:
- note added: "150mA LDO"
- note removed: "500mA LDO"
- moved on the sheet: C22, C23, C24, C25, C26, C27, C28, C29, C31, C32, C33, U14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

Commit message: fix
Parts:
- removed U15: CJT1117-3.3, Package_TO_SOT_SMD:SOT-223, symbol Ninja-qPCR:CJT1117-3.3
- removed U16: CJT1117-5.0, Package_TO_SOT_SMD:SOT-223, symbol Ninja-qPCR:CJT1117-3.3
- added U3: BD433M5FP-CE2, Ninja-qPCR:REG_TO252-3, symbol Ninja-qPCR:REG_TO252-3
- added U6: BA178M05FP-E2, Ninja-qPCR:REG_TO252-3, symbol Ninja-qPCR:REG_TO252-3
Connections:
- net 20V: now also U3.1 (VIN), U6.1 (VIN)
- net 3V3D: now also U3.2 (VOUT)
- net 5V: now also U6.2 (VOUT)
- net GND: now also U3.3 (GND), U6.3 (GND)
Changed lines of the file:
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@@
-    (stroke (width 0) (type default) (color 0 0 0 0))
-  )
-  (wire (pts (xy 244.475 73.025) (xy 240.665 73.025))
     (stroke (width 0) (type default) (color 0 0 0 0))
   )
@@
     (stroke (width 0) (type default) (color 0 0 0 0))
   )
+  (wire (pts (xy 212.725 43.815) (xy 220.345 43.815))
+    (stroke (width 0) (type default) (color 0 0 0 0))
+  )
   (wire (pts (xy 105.41 124.46) (xy 102.87 124.46))
     (stroke (width 0) (type default) (color 0 0 0 0))
@@
     (stroke (width 0) (type default) (color 0 0 0 0))
   )
-  (wire (pts (xy 216.535 75.565) (xy 216.535 78.105))
+  (wire (pts (xy 229.235 80.645) (xy 229.235 83.185))
     (stroke (width 0) (type default) (color 0 0 0 0))
   )
@@
     (stroke (width 0) (type default) (color 0 0 0 0))
   )
-  (wire (pts (xy 244.475 43.815) (xy 240.665 43.815))
+  (wire (pts (xy 238.125 43.815) (xy 244.475 43.815))
     (stroke (width 0) (type default) (color 0 0 0 0))
   )
@@
     (stroke (width 0) (type default) (color 0 0 0 0))
   )
-  (wire (pts (xy 219.075 46.355) (xy 216.535 46.355))
-    (stroke (width 0) (type default) (color 0 0 0 0))
-  )
   (wire (pts (xy 255.905 43.815) (xy 255.905 50.165))
     (stroke (width 0) (type default) (color 0 0 0 0))
@@
     (stroke (width 0) (type default) (color 0 0 0 0))
   )
+  (wire (pts (xy 238.125 73.025) (xy 244.475 73.025))
+    (stroke (width 0) (type default) (color 0 0 0 0))
+  )
   (wire (pts (xy 88.9 44.45) (xy 92.71 44.45))
     (stroke (width 0) (type default) (color 0 0 0 0))
@@
     (stroke (width 0) (type default) (color 0 0 0 0))
   )
-  (wire (pts (xy 219.075 75.565) (xy 216.535 75.565))
-    (stroke (width 0) (type default) (color 0 0 0 0))
-  )
   (wire (pts (xy 45.72 60.96) (xy 45.72 58.42))
     (stroke (width 0) (type default) (color 0 0 0 0))
@@
     (stroke (width 0) (type default) (color 0 0 0 0))
   )
-  (wire (pts (xy 216.535 46.355) (xy 216.535 48.895))
+  (wire (pts (xy 229.235 51.435) (xy 229.235 53.975))
     (stroke (width 0) (type default) (color 0 0 0 0))
   )
@@
     (stroke (width 0) (type default) (color 0 0 0 0))
   )
-  (wire (pts (xy 219.075 43.815) (xy 212.725 43.815))
-    (stroke (width 0) (type default) (color 0 0 0 0))
-  )
   (wire (pts (xy 203.835 43.815) (xy 203.835 50.165))
     (stroke (width 0) (type default) (color 0 0 0 0))
@@
     (stroke (width 0) (type default) (color 0 0 0 0))
   )
-  (wire (pts (xy 212.725 73.025) (xy 219.075 73.025))
+  (wire (pts (xy 212.725 73.025) (xy 220.345 73.025))
     (stroke (width 0) (type default) (color 0 0 0 0))
   )
@@
     )
     (pin "1")
+  )
+  (symbol (lib_id "Ninja-qPCR:REG_TO252-3") (at 229.235 71.755 0) (unit 1)
+    (in_bom yes) (on_board yes)
+    (property "Reference" "U6" (id 0) (at 228.6 68.58 0))
+    (property "Value" "BA178M05FP-E2" (id 1) (at 229.235 70.485 0))
+    (property "Footprint" "Ninja-qPCR:REG_TO252-3" (id 2) (at 227.965 70.485 0)
+      (effects (font (size 1.27 1.27)) hide)
+    )
+    (property "Datasheet" "" (id 3) (at 227.965 70.485 0)
+      (effects (font (size 1.27 1.27)) hide)
+    )
+    (pin "1")
+    (pin "2")
+    (pin "3")
   )
   (symbol (lib_id "power:GND") (at 192.405 61.595 0) (unit 1)
@@
     (pin "1")
   )
+  (symbol (lib_id "Ninja-qPCR:REG_TO252-3") (at 229.235 42.545 0) (unit 1)
+    (in_bom yes) (on_board yes)
+    (property "Reference" "U3" (id 0) (at 229.235 38.735 0))
+    (property "Value" "BD433M5FP-CE2" (id 1) (at 229.87 41.275 0))
+    (property "Footprint" "Ninja-qPCR:REG_TO252-3" (id 2) (at 227.965 41.275 0)
+      (effects (font (size 1.27 1.27)) hide)
+    )
+    (property "Datasheet" "" (id 3) (at 227.965 41.275 0)
+      (effects (font (size 1.27 1.27)) hide)
+    )
+    (pin "1")
+    (pin "2")
+    (pin "3")
+  )
   (symbol (lib_id "power:GND") (at 244.475 90.805 0) (unit 1)
     (in_bom yes) (on_board yes)
@@
     (pin "1")
   )
-  (symbol (lib_id "power:GND") (at 216.535 78.105 0) (unit 1)
-    (in_bom yes) (on_board yes)
-    (property "Reference" "#PWR0132" (id 0) (at 216.535 84.455 0)
-      (effects (font (size 1.27 1.27)) hide)
-    )
-    (property "Value" "GND" (id 1) (at 216.662 82.4992 0))
-    (property "Footprint" "" (id 2) (at 216.535 78.105 0)
-      (effects (font (size 1.27 1.27)) hide)
-    )
-    (property "Datasheet" "" (id 3) (at 216.535 78.105 0)
+  (symbol (lib_id "power:GND") (at 229.235 83.185 0) (unit 1)
+    (in_bom yes) (on_board yes)
+    (property "Reference" "#PWR0132" (id 0) (at 229.235 89.535 0)
+      (effects (font (size 1.27 1.27)) hide)
+    )
+    (property "Value" "GND" (id 1) (at 229.362 87.5792 0))
+    (property "Footprint" "" (id 2) (at 229.235 83.185 0)
+      (effects (font (size 1.27 1.27)) hide)
+    )
+    (property "Datasheet" "" (id 3) (at 229.235 83.185 0)
       (effects (font (size 1.27 1.27)) hide)
     )
@@
     (pin "1")
   )
-  (symbol (lib_id "power:GND") (at 216.535 48.895 0) (unit 1)
-    (in_bom yes) (on_board yes)
-    (property "Reference" "#PWR0133" (id 0) (at 216.535 55.245 0)
-      (effects (font (size 1.27 1.27)) hide)
-    )
-    (property "Value" "GND" (id 1) (at 216.662 53.2892 0))
-    (property "Footprint" "" (id 2) (at 216.535 48.895 0)
-      (effects (font (size 1.27 1.27)) hide)
-    )
-    (property "Datasheet" "" (id 3) (at 216.535 48.895 0)
+  (symbol (lib_id "power:GND") (at 229.235 53.975 0) (unit 1)
+    (in_bom yes) (on_board yes)
+    (property "Reference" "#PWR0133" (id 0) (at 229.235 60.325 0)
+      (effects (font (size 1.27 1.27)) hide)
+    )
+    (property "Value" "GND" (id 1) (at 229.362 58.3692 0))
+    (property "Footprint" "" (id 2) (at 229.235 53.975 0)
+      (effects (font (size 1.27 1.27)) hide)
+    )
+    (property "Datasheet" "" (id 3) (at 229.235 53.975 0)
       (effects (font (size 1.27 1.27)) hide)
     )
@@
     (pin "2")
   )
-  (symbol (lib_id "Ninja-qPCR:CJT1117-3.3") (at 229.235 71.755 0) (unit 1)
-    (in_bom yes) (on_board yes)
-    (property "Reference" "U16" (id 0) (at 229.87 67.31 0))
-    (property "Value" "CJT1117-5.0" (id 1) (at 229.87 69.6214 0))
-    (property "Footprint" "Package_TO_SOT_SMD:SOT-223" (id 2) (at 229.235 73.025 0)
-      (effects (font (size 1.27 1.27)) hide)
-    )
-    (property "Datasheet" "" (id 3) (at 229.235 73.025 0)
-      (effects (font (size 1.27 1.27)) hide)
-    )
-    (pin "1")
-    (pin "2")
-    (pin "3")
-    (pin "4")
-  )
   (symbol (lib_id "Device:R") (at 124.46 49.53 180) (unit 1)
     (in_bom yes) (on_board yes)
@@
     (pin "2")
   )
-  (symbol (lib_id "Ninja-qPCR:CJT1117-3.3") (at 229.235 42.545 0) (unit 1)
-    (in_bom yes) (on_board yes)
-    (property "Reference" "U15" (id 0) (at 229.87 38.1 0))
-    (property "Value" "CJT1117-3.3" (id 1) (at 229.87 40.4114 0))
-    (property "Footprint" "Package_TO_SOT_SMD:SOT-223" (id 2) (at 229.235 43.815 0)
-      (effects (font (size 1.27 1.27)) hide)
-    )
-    (property "Datasheet" "" (id 3) (at 229.235 43.815 0)
-      (effects (font (size 1.27 1.27)) hide)
-    )
-    (pin "1")
-    (pin "2")
-    (pin "3")
-    (pin "4")
-  )
 )

Commit message: sync
Parts:
- removed C14, C16: 1uF, Capacitor_SMD:C_0603_1608Metric, symbol Device:C
- removed C19: 10uF, Capacitor_SMD:C_0805_2012Metric, symbol Device:C
- removed C20, C21: 22uF, Capacitor_SMD:C_1210_3225Metric, symbol Device:C
- removed R15: 150k, Resistor_SMD:R_0603_1608Metric, symbol Device:R
- removed U12: TPS63710DRRR, Ninja-qPCR:TPS63710DRRR, symbol Ninja-qPCR:TPS63710DRRR
- added C2: 0.1uF, Capacitor_SMD:C_0603_1608Metric, symbol Device:C
- added C7: 22uF, Capacitor_SMD:C_1210_3225Metric, symbol Device:C
- added U7: AZ34063U, Package_SO:SOP-8_3.9x4.9mm_P1.27mm, symbol Ninja-qPCR:AZ34063U
- L1: value 2.2uH -> 68uH; footprint Capacitor_SMD:C_0805_2012Metric -> (none)
- R5: value 39k -> 0.24
Connections:
- net -1V: now also C2.2, C7.2, U7.4 (GND); no longer L1.2
- net 3V3D: now also R5.2, U7.6 (VCC); no longer C15.1
- net GND: now also C7.1, U7.5 (COMP)
- net at R5.1: now also U7.1 (SC), U7.7 (SENSE), U7.8 (DC)
- net at L1.1: now also U7.2 (SE)
- new net: C2.1, U7.3 (TC)
- no-connect marks 2 -> 1
Other:
- moved on the sheet: C12, C15

Commit message: sync
Parts:
- added D1: D_Schottky, Ninja-qPCR:MSS1P3L-M3&slash_89A, symbol Device:D_Schottky
- L1: footprint (none) -> Inductor_SMD:L_Taiyo-Yuden_NR-60xx
Connections:
- net -1V: now also D1.2 (A)
- net 3V3D: now also C15.1
- net GND: now also L1.2
- net at L1.1, U7.2 (SE): now also D1.1 (K)
Other:
- moved on the sheet: C7, L1

Commit message: ordered batch2/main
Parts:
- removed C12, C7: 22uF, Capacitor_SMD:C_1210_3225Metric, symbol Device:C
- removed C15: 1uF, Capacitor_SMD:C_0603_1608Metric, symbol Device:C
- removed C2: 0.1uF, Capacitor_SMD:C_0603_1608Metric, symbol Device:C
- removed D1: D_Schottky, Ninja-qPCR:MSS1P3L-M3&slash_89A, symbol Device:D_Schottky
- removed L1: 68uH, Inductor_SMD:L_Taiyo-Yuden_NR-60xx, symbol Device:L
- removed R5: 0.24, Resistor_SMD:R_0603_1608Metric, symbol Device:R
- removed U7: AZ34063U, Package_SO:SOP-8_3.9x4.9mm_P1.27mm, symbol Ninja-qPCR:AZ34063U
- added C16: 0.1uF, Capacitor_SMD:C_0603_1608Metric, symbol Device:C
- added C19: 3300pF, Capacitor_SMD:C_0603_1608Metric, symbol Device:C
- added C20, C21: 10uF, Capacitor_SMD:C_0805_2012Metric, symbol Device:C
- added D2, D3: D_Schottky, Ninja-qPCR:MSS1P3L-M3&slash_89A, symbol Device:D_Schottky
- added J4, J5: Conn_01x02_Male, Connector_PinHeader_1.27mm:PinHeader_1x02_P1.27mm_Vertical, symbol Connector:Conn_01x02_Male
- added JP4: Jumper_3_Open, Jumper:SolderJumper-3_P2.0mm_Open_TrianglePad1.0x1.5mm, symbol Jumper:Jumper_3_Open
- added R14: 0.1k, Resistor_SMD:R_0603_1608Metric, symbol Device:R
- added R15, R25: 10k, Resistor_SMD:R_0603_1608Metric, symbol Device:R
- added R24: 51k, Resistor_SMD:R_0603_1608Metric, symbol Device:R
- added U12: NE555, Package_SO:SOIC-8_3.9x4.9mm_P1.27mm, symbol Ninja-qPCR:NE555
- added U13: LM393, Package_SO:SOIC-8_3.9x4.9mm_P1.27mm, symbol Comparator:LM393
Connections:
- net -1V: now also C21.1, D3.2 (A), J5.2 (Pin_2), R25.1
- net 3V3D: now also C16.1, J4.1 (Pin_1), R14.1, R24.2, U12.8 (Vcc), U13.8 (V+)
- net 5V: now also C22.1, C24.1, C26.1, U14.1 (VIN), U14.3 (SHDN)
- net GND: now also C16.2, C19.2, C21.2, D2.1 (K), U12.1 (GND), U13.2 (-), U13.4 (V-)
- new net: JP4.3 (B), R24.1, R25.2
- new net: R14.2, R15.1, U12.7 (DISCH)
- new net: C19.1, R15.2, U12.2 (TRIG), U12.6 (THRES)
- new net: C20.1, D2.2 (A), D3.1 (K)
- new net: C20.2, U12.3 (OUT)
- new net: JP4.2 (C), U13.3 (+)
- new net: J4.2 (Pin_2), J5.1 (Pin_1), JP4.1 (A)
- new net RST-1V: U12.4 (RESET), U13.1
- no-connect marks 1 -> 2
Other:
- moved on the sheet: J2
