File: kicad/NinjaLite/batch03/main/_autosave-filePhoto.kicad_sch (KiCad schematic)
At the start: 22 parts, among them J13 Conn_01x01_Male, J16 Conn_01x01_Male, J23 Conn_01x01_Male, J24 Conn_01x02_Male, J25 Conn_01x02_Male, J26 Conn_01x02_Male, J27 Conn_01x02_Male, J4 Conn_01x02_Male, U1 NAU7802, U2 NAU7802, U4 LMP7717MF_NOPB

Commit message: just before ripup batch03/main
Parts:
- gave numbers to parts that had none: 1
Changed lines of the file:
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@@
   (symbol (lib_id "Device:R") (at 173.99 50.292 90) (mirror x) (unit 1)
     (in_bom yes) (on_board yes)
-    (property "Reference" "R?" (id 0) (at 173.99 45.0342 90))
+    (property "Reference" "R5" (id 0) (at 173.99 45.0342 90))
     (property "Value" "10M" (id 1) (at 173.99 47.3456 90))
     (property "Footprint" "Resistor_SMD:R_0603_1608Metric" (id 2) (at 173.99 48.514 90)
