File: kicad/NinjaLite/batch03/main/filePhoto.kicad_sch (KiCad schematic)
At the start: 22 parts, among them J13 Conn_01x01_Male, J16 Conn_01x01_Male, J23 Conn_01x01_Male, J24 Conn_01x02_Male, J25 Conn_01x02_Male, J26 Conn_01x02_Male, J27 Conn_01x02_Male, J4 Conn_01x02_Male, U1 NAU7802, U2 NAU7802, U4 LMP7717MF_NOPB

Commit message: wiring batch03/main
Parts:
- gave numbers to parts that had none: 1
Connections:
- net AMP_OUT: now also JP6.2 (C); no longer C6.1, J4.2 (Pin_2), JP6.1 (A), R13.2
- net PD_MUX_OUT: now also J24.1 (Pin_1), J25.1 (Pin_1)
- new net: C6.1, J4.2 (Pin_2), JP6.1 (A), R13.2
Changed lines of the file:
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@@
   (junction (at 81.407 102.362) (diameter 0) (color 0 0 0 0)
   )
+  (junction (at 182.245 39.497) (diameter 0) (color 0 0 0 0)
+  )
+  (junction (at 244.475 62.23) (diameter 0) (color 0 0 0 0)
+  )
+  (junction (at 191.77 37.592) (diameter 0) (color 0 0 0 0)
+  )
   (junction (at 163.576 50.292) (diameter 0) (color 0 0 0 0)
   )
-  (junction (at 244.475 62.23) (diameter 0) (color 0 0 0 0)
-  )
-  (junction (at 205.74 50.292) (diameter 0) (color 0 0 0 0)
-  )
-  (junction (at 191.77 37.592) (diameter 0) (color 0 0 0 0)
-  )
   (junction (at 81.407 57.15) (diameter 0) (color 0 0 0 0)
   )
@@
   (junction (at 111.887 81.28) (diameter 0) (color 0 0 0 0)
   )
+  (junction (at 223.52 43.942) (diameter 0) (color 0 0 0 0)
+  )
   (junction (at 167.132 50.292) (diameter 0) (color 0 0 0 0)
   )
-  (junction (at 182.372 39.37) (diameter 0) (color 0 0 0 0)
-  )
   (junction (at 223.52 97.536) (diameter 0) (color 0 0 0 0)
   )
   (junction (at 111.887 68.58) (diameter 0) (color 0 0 0 0)
-  )
-  (junction (at 223.52 50.292) (diameter 0) (color 0 0 0 0)
   )
   (junction (at 208.28 91.44) (diameter 0) (color 0 0 0 0)
@@
     (stroke (width 0) (type default) (color 0 0 0 0))
   )
-  (wire (pts (xy 205.74 50.292) (xy 223.52 50.292))
-    (stroke (width 0) (type default) (color 0 0 0 0))
-  )
   (wire (pts (xy 208.28 97.536) (xy 223.52 97.536))
     (stroke (width 0) (type default) (color 0 0 0 0))
@@
     (stroke (width 0) (type default) (color 0 0 0 0))
   )
+  (wire (pts (xy 182.245 39.497) (xy 163.576 39.497))
+    (stroke (width 0) (type default) (color 0 0 0 0))
+  )
   (wire (pts (xy 80.137 57.15) (xy 81.407 57.15))
     (stroke (width 0) (type default) (color 0 0 0 0))
@@
     (stroke (width 0) (type default) (color 0 0 0 0))
   )
-  (wire (pts (xy 223.52 50.292) (xy 223.52 81.28))
+  (wire (pts (xy 223.52 43.942) (xy 223.52 81.28))
     (stroke (width 0) (type default) (color 0 0 0 0))
   )
@@
     (stroke (width 0) (type default) (color 0 0 0 0))
   )
+  (wire (pts (xy 209.55 43.942) (xy 223.52 43.942))
+    (stroke (width 0) (type default) (color 0 0 0 0))
+  )
   (wire (pts (xy 184.785 37.592) (xy 184.785 32.512))
     (stroke (width 0) (type default) (color 0 0 0 0))
@@
     (stroke (width 0) (type default) (color 0 0 0 0))
   )
-  (wire (pts (xy 163.576 39.37) (xy 163.576 50.292))
-    (stroke (width 0) (type default) (color 0 0 0 0))
-  )
   (wire (pts (xy 244.475 62.23) (xy 263.525 62.23))
     (stroke (width 0) (type default) (color 0 0 0 0))
@@
     (stroke (width 0) (type default) (color 0 0 0 0))
   )
-  (wire (pts (xy 182.372 39.37) (xy 163.576 39.37))
-    (stroke (width 0) (type default) (color 0 0 0 0))
-  )
   (wire (pts (xy 56.642 80.01) (xy 61.087 80.01))
     (stroke (width 0) (type default) (color 0 0 0 0))
@@
     (stroke (width 0) (type default) (color 0 0 0 0))
   )
-  (wire (pts (xy 223.52 50.292) (xy 224.79 50.292))
+  (wire (pts (xy 223.52 43.942) (xy 224.79 43.942))
     (stroke (width 0) (type default) (color 0 0 0 0))
   )
@@
   )
   (wire (pts (xy 244.475 62.23) (xy 244.475 67.31))
+    (stroke (width 0) (type default) (color 0 0 0 0))
+  )
+  (wire (pts (xy 163.576 39.497) (xy 163.576 50.292))
     (stroke (width 0) (type default) (color 0 0 0 0))
   )
@@
     (effects (font (size 1.27 1.27)) (justify right))
   )
-  (hierarchical_label "AMP_OUT" (shape input) (at 224.79 50.292 0)
+  (hierarchical_label "AMP_OUT" (shape input) (at 224.79 43.942 0)
     (effects (font (size 1.27 1.27)) (justify left))
   )
@@
   (symbol (lib_id "Device:R") (at 173.99 50.292 90) (mirror x) (unit 1)
     (in_bom yes) (on_board yes)
-    (property "Reference" "R?" (id 0) (at 173.99 45.0342 90))
+    (property "Reference" "R5" (id 0) (at 173.99 45.0342 90))
     (property "Value" "10M" (id 1) (at 173.99 47.3456 90))
     (property "Footprint" "Resistor_SMD:R_0603_1608Metric" (id 2) (at 173.99 48.514 90)
