File: kicad/NinjaLite/batch03/main/filePhotoThermistors.kicad_sch (KiCad schematic)
At the start: 10 parts, among them U8 TS12A12511DCNR, U9 SN74LV4051A

Commit message: wiring batch03/main done
Parts:
- TEXT1, TEXT2, TEXT3: footprint Connector_PinHeader_2.54mm:PinHeader_1x02_P2.54mm_Vertical -> Pin_Headers:Pin_Header_Straight_1x02_Pitch1.27mm
- TLID1, TWELL1: footprint Connector_PinHeader_2.54mm:PinHeader_1x02_P2.54mm_Vertical -> Connector_Hirose:Hirose_DF13-02P-1.25DSA_1x02_P1.25mm_Vertical
Changed lines of the file:
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@@
     (property "Reference" "TEXT1" (id 0) (at 257.81 80.01 0))
     (property "Value" "Conn_01x02_Male" (id 1) (at 264.16 82.55 0))
-    (property "Footprint" "Connector_PinHeader_2.54mm:PinHeader_1x02_P2.54mm_Vertical" (id 2) (at 254 80.01 0)
+    (property "Footprint" "Pin_Headers:Pin_Header_Straight_1x02_Pitch1.27mm" (id 2) (at 254 80.01 0)
       (effects (font (size 1.27 1.27)) hide)
     )
@@
     (property "Reference" "TLID1" (id 0) (at 257.81 64.77 0))
     (property "Value" "Conn_01x02_Male" (id 1) (at 264.16 67.31 0))
-    (property "Footprint" "Connector_PinHeader_2.54mm:PinHeader_1x02_P2.54mm_Vertical" (id 2) (at 254 64.77 0)
+    (property "Footprint" "Connector_Hirose:Hirose_DF13-02P-1.25DSA_1x02_P1.25mm_Vertical" (id 2) (at 254 64.77 0)
       (effects (font (size 1.27 1.27)) hide)
     )
@@
     (property "Reference" "TEXT2" (id 0) (at 257.81 88.9 0))
     (property "Value" "Conn_01x02_Male" (id 1) (at 264.16 91.44 0))
-    (property "Footprint" "Connector_PinHeader_2.54mm:PinHeader_1x02_P2.54mm_Vertical" (id 2) (at 254 88.9 0)
+    (property "Footprint" "Pin_Headers:Pin_Header_Straight_1x02_Pitch1.27mm" (id 2) (at 254 88.9 0)
       (effects (font (size 1.27 1.27)) hide)
     )
@@
     (property "Reference" "TWELL1" (id 0) (at 257.81 49.53 0))
     (property "Value" "Conn_01x02_Male" (id 1) (at 264.16 52.07 0))
-    (property "Footprint" "Connector_PinHeader_2.54mm:PinHeader_1x02_P2.54mm_Vertical" (id 2) (at 254 49.53 0)
+    (property "Footprint" "Connector_Hirose:Hirose_DF13-02P-1.25DSA_1x02_P1.25mm_Vertical" (id 2) (at 254 49.53 0)
       (effects (font (size 1.27 1.27)) hide)
     )
@@
     (property "Reference" "TEXT3" (id 0) (at 257.81 96.52 0))
     (property "Value" "Conn_01x02_Male" (id 1) (at 264.16 99.06 0))
-    (property "Footprint" "Connector_PinHeader_2.54mm:PinHeader_1x02_P2.54mm_Vertical" (id 2) (at 254 96.52 0)
+    (property "Footprint" "Pin_Headers:Pin_Header_Straight_1x02_Pitch1.27mm" (id 2) (at 254 96.52 0)
       (effects (font (size 1.27 1.27)) hide)
     )
