File: kicad/NinjaLite/batch03/main/qLAMP-main.kicad_sch (KiCad schematic)
At the start: 17 parts, among them J3 Conn_01x07_Male, Q3 Q_NMOS_GSD, Q5 Q_NMOS_GSD, U17 LITE_LCD, U5 ESP32-WROOM-32

Commit message: just before ripup batch03/main
Connections:
- net 20V renamed VCC

Commit message: wiring batch03/main done
Parts:
- added J5, J6, J7: Conn_01x01_Male, Pin_Headers:Pin_Header_Straight_1x01_Pitch1.27mm, symbol Connector:Conn_01x01_Male
Connections:
- net at U5.6 (IO34): now also J6.1 (Pin_1)
- net at U5.7 (IO35): now also J7.1 (Pin_1)
- net ADC_DRDY: no longer names the net of U5.28 (IO17)
- net ADC_DRDY: now also J5.1 (Pin_1)
- no-connect marks 6 -> 4
Changed lines of the file:
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@@
   (no_connect (at 54.61 173.355))
   (no_connect (at 54.61 163.195))
-  (no_connect (at 67.31 125.73))
-  (no_connect (at 67.31 128.27))
   (wire (pts (xy 71.12 69.85) (xy 88.9 69.85))
     (stroke (width 0) (type default) (color 0 0 0 0))
@@
     (stroke (width 0) (type default) (color 0 0 0 0))
   )
-  (wire (pts (xy 63.5 128.27) (xy 67.31 128.27))
-    (stroke (width 0) (type default) (color 0 0 0 0))
-  )
   (wire (pts (xy 48.26 52.07) (xy 48.26 64.77))
     (stroke (width 0) (type default) (color 0 0 0 0))
@@
     (stroke (width 0) (type default) (color 0 0 0 0))
   )
-  (wire (pts (xy 63.5 125.73) (xy 67.31 125.73))
+  (wire (pts (xy 63.5 125.73) (xy 79.248 125.73))
     (stroke (width 0) (type default) (color 0 0 0 0))
   )
@@
     (stroke (width 0) (type default) (color 0 0 0 0))
   )
-  (wire (pts (xy 63.5 97.79) (xy 67.31 97.79))
+  (wire (pts (xy 63.5 97.79) (xy 79.248 97.79))
     (stroke (width 0) (type default) (color 0 0 0 0))
   )
@@
   )
   (wire (pts (xy 220.98 138.43) (xy 224.79 138.43))
+    (stroke (width 0) (type default) (color 0 0 0 0))
+  )
+  (wire (pts (xy 63.5 128.27) (xy 79.248 128.27))
     (stroke (width 0) (type default) (color 0 0 0 0))
   )
@@
     (effects (font (size 1.27 1.27)) (justify left bottom))
   )
-  (text "NOT IN USE YET (IO34-39 INPUT ONLY)" (at 68.58 128.905 0)
+  (text "NOT IN USE YET (IO34-39 INPUT ONLY)" (at 68.326 131.699 0)
     (effects (font (size 1.27 1.27)) (justify left bottom))
   )
@@
     (property "Intersheet References" "${INTERSHEET_REFS}" (id 0) (at 201.0572 65.9606 0)
       (effects (font (size 1.27 1.27)) (justify right) hide)
-    )
-  )
-  (global_label "ADC_DRDY" (shape input) (at 67.31 97.79 0) (fields_autoplaced)
-    (effects (font (size 1.27 1.27)) (justify left))
-    (property "Intersheet References" "${INTERSHEET_REFS}" (id 0) (at 79.129 97.7106 0)
-      (effects (font (size 1.27 1.27)) (justify left) hide)
     )
   )
@@
     (pin "1")
   )
+  (symbol (lib_id "Connector:Conn_01x01_Male") (at 84.328 128.27 0) (mirror y) (unit 1)
+    (in_bom yes) (on_board yes) (fields_autoplaced)
+    (property "Reference" "J7" (id 0) (at 83.693 124.494 0))
+    (property "Value" "Conn_01x01_Male" (id 1) (at 83.693 127.0309 0))
+    (property "Footprint" "Pin_Headers:Pin_Header_Straight_1x01_Pitch1.27mm" (id 2) (at 84.328 128.27 0)
+      (effects (font (size 1.27 1.27)) hide)
+    )
+    (property "Datasheet" "~" (id 3) (at 84.328 128.27 0)
+      (effects (font (size 1.27 1.27)) hide)
+    )
+    (pin "1")
+  )
   (symbol (lib_id "Device:R") (at 22.86 59.69 180) (unit 1)
     (in_bom yes) (on_board yes)
@@
     (pin "1")
     (pin "2")
+  )
+  (symbol (lib_id "Connector:Conn_01x01_Male") (at 84.328 125.73 0) (mirror y) (unit 1)
+    (in_bom yes) (on_board yes) (fields_autoplaced)
+    (property "Reference" "J6" (id 0) (at 83.693 121.954 0))
+    (property "Value" "Conn_01x01_Male" (id 1) (at 83.693 124.4909 0))
+    (property "Footprint" "Pin_Headers:Pin_Header_Straight_1x01_Pitch1.27mm" (id 2) (at 84.328 125.73 0)
+      (effects (font (size 1.27 1.27)) hide)
+    )
+    (property "Datasheet" "~" (id 3) (at 84.328 125.73 0)
+      (effects (font (size 1.27 1.27)) hide)
+    )
+    (pin "1")
   )
   (symbol (lib_id "Device:C") (at 22.86 76.2 0) (unit 1)
@@
     (pin "9")
   )
+  (symbol (lib_id "Connector:Conn_01x01_Male") (at 84.328 97.79 0) (mirror y) (unit 1)
+    (in_bom yes) (on_board yes) (fields_autoplaced)
+    (property "Reference" "J5" (id 0) (at 83.693 94.014 0))
+    (property "Value" "Conn_01x01_Male" (id 1) (at 83.693 96.5509 0))
+    (property "Footprint" "Pin_Headers:Pin_Header_Straight_1x01_Pitch1.27mm" (id 2) (at 84.328 97.79 0)
+      (effects (font (size 1.27 1.27)) hide)
+    )
+    (property "Datasheet" "~" (id 3) (at 84.328 97.79 0)
+      (effects (font (size 1.27 1.27)) hide)
+    )
+    (pin "1")
+  )
   (symbol (lib_id "Device:R") (at 86.36 59.69 180) (unit 1)
     (in_bom yes) (on_board yes)
@@
       (reference "J4") (unit 1) (value "Conn_01x02_Male") (footprint "Connector_PinHeader_2.54mm:PinHeader_1x02_P2.54mm_Vertical")
     )
+    (path "/b0df3198-4f99-47c8-a1ce-4ac585098c18"
+      (reference "J5") (unit 1) (value "Conn_01x01_Male") (footprint "Pin_Headers:Pin_Header_Straight_1x01_Pitch1.27mm")
+    )
+    (path "/6eab180f-5d09-4f6e-b931-59ed96c65357"
+      (reference "J6") (unit 1) (value "Conn_01x01_Male") (footprint "Pin_Headers:Pin_Header_Straight_1x01_Pitch1.27mm")
+    )
+    (path "/57b496f8-9a08-4ec2-bf0c-790596dc5d8a"
+      (reference "J7") (unit 1) (value "Conn_01x01_Male") (footprint "Pin_Headers:Pin_Header_Straight_1x01_Pitch1.27mm")
+    )
     (path "/00000000-0000-0000-0000-0000614a3cbb/00000000-0000-0000-0000-0000614d4c2b"
       (reference "J13") (unit 1) (value "Conn_01x01_Male") (footprint "Connector_PinHeader_1.27mm:PinHeader_1x01_P1.27mm_Vertical")
@@
     )
     (path "/00000000-0000-0000-0000-0000614a49f9/00000000-0000-0000-0000-000060e1fb7c"
-      (reference "TEXT1") (unit 1) (value "Conn_01x02_Male") (footprint "Connector_PinHeader_2.54mm:PinHeader_1x02_P2.54mm_Vertical")
+      (reference "TEXT1") (unit 1) (value "Conn_01x02_Male") (footprint "Pin_Headers:Pin_Header_Straight_1x02_Pitch1.27mm")
     )
     (path "/00000000-0000-0000-0000-0000614a49f9/00000000-0000-0000-0000-000060e1fb8e"
-      (reference "TEXT2") (unit 1) (value "Conn_01x02_Male") (footprint "Connector_PinHeader_2.54mm:PinHeader_1x02_P2.54mm_Vertical")
+      (reference "TEXT2") (unit 1) (value "Conn_01x02_Male") (footprint "Pin_Headers:Pin_Header_Straight_1x02_Pitch1.27mm")
     )
     (path "/00000000-0000-0000-0000-0000614a49f9/00000000-0000-0000-0000-000060e2b42c"
-      (reference "TEXT3") (unit 1) (value "Conn_01x02_Male") (footprint "Connector_PinHeader_2.54mm:PinHeader_1x02_P2.54mm_Vertical")
+      (reference "TEXT3") (unit 1) (value "Conn_01x02_Male") (footprint "Pin_Headers:Pin_Header_Straight_1x02_Pitch1.27mm")
     )
     (path "/00000000-0000-0000-0000-0000614a49f9/00000000-0000-0000-0000-000060e1fb82"
-      (reference "TLID1") (unit 1) (value "Conn_01x02_Male") (footprint "Connector_PinHeader_2.54mm:PinHeader_1x02_P2.54mm_Vertical")
+      (reference "TLID1") (unit 1) (value "Conn_01x02_Male") (footprint "Connector_Hirose:Hirose_DF13-02P-1.25DSA_1x02_P1.25mm_Vertical")
     )
     (path "/00000000-0000-0000-0000-0000614a49f9/00000000-0000-0000-0000-000060e2ab80"
-      (reference "TWELL1") (unit 1) (value "Conn_01x02_Male") (footprint "Connector_PinHeader_2.54mm:PinHeader_1x02_P2.54mm_Vertical")
+      (reference "TWELL1") (unit 1) (value "Conn_01x02_Male") (footprint "Connector_Hirose:Hirose_DF13-02P-1.25DSA_1x02_P1.25mm_Vertical")
     )
     (path "/00000000-0000-0000-0000-0000614a3cbb/7f1ae94a-6efa-44d9-baeb-70b779540721"
