File: kicad/NinjaLite/batch03/main-pdb/filePower.kicad_sch (KiCad schematic)
At the start: 27 parts, among them J1 ALI_USB, J2 Barrel_Jack_Switch, Q1 Q_NMOS_GSD, U11 IP2721, U14 TCR3DF33,LM(CT, U3 BD433M5FP-CE2, U6 BA178M05FP-E2

Commit message: add reg alt
Parts:
- added U12, U7: LD1086DTTR, Package_TO_SOT_SMD:SOT-223, symbol Regulator_Linear:LD1086DTTR
Connections:
- net 3V3D: now also U12.2 (OUT)
- net 5V: now also U7.2 (OUT)
- net GND: now also U12.1 (ADJ/GND), U7.1 (ADJ/GND)
- net VCC: now also U12.3 (IN), U7.3 (IN)
Changed lines of the file:
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@@
+    (stroke (width 0) (type default) (color 0 0 0 0))
+  )
+  (wire (pts (xy 136.906 111.76) (xy 138.43 111.76))
     (stroke (width 0) (type default) (color 0 0 0 0))
   )
@@
     (stroke (width 0) (type default) (color 0 0 0 0))
   )
+  (wire (pts (xy 114.3 111.76) (xy 116.586 111.76))
+    (stroke (width 0) (type default) (color 0 0 0 0))
+  )
   (wire (pts (xy 53.34 76.2) (xy 53.34 78.74))
     (stroke (width 0) (type default) (color 0 0 0 0))
@@
     (stroke (width 0) (type default) (color 0 0 0 0))
   )
+  (wire (pts (xy 126.746 119.38) (xy 126.746 120.904))
+    (stroke (width 0) (type default) (color 0 0 0 0))
+  )
   (wire (pts (xy 154.94 171.45) (xy 154.94 173.99))
     (stroke (width 0) (type default) (color 0 0 0 0))
@@
     (stroke (width 0) (type default) (color 0 0 0 0))
   )
+  (wire (pts (xy 76.708 111.76) (xy 78.994 111.76))
+    (stroke (width 0) (type default) (color 0 0 0 0))
+  )
   (wire (pts (xy 60.96 66.04) (xy 60.96 68.58))
     (stroke (width 0) (type default) (color 0 0 0 0))
@@
     (stroke (width 0) (type default) (color 0 0 0 0))
   )
+  (wire (pts (xy 89.154 119.38) (xy 89.154 120.904))
+    (stroke (width 0) (type default) (color 0 0 0 0))
+  )
   (wire (pts (xy 53.34 63.5) (xy 66.04 63.5))
     (stroke (width 0) (type default) (color 0 0 0 0))
@@
   )
   (wire (pts (xy 203.835 57.785) (xy 203.835 61.595))
+    (stroke (width 0) (type default) (color 0 0 0 0))
+  )
+  (wire (pts (xy 99.314 111.76) (xy 100.838 111.76))
     (stroke (width 0) (type default) (color 0 0 0 0))
   )
@@
     (property "Intersheet References" "${INTERSHEET_REFS}" (id 0) (at 80.645 -61.595 0)
       (effects (font (size 1.27 1.27)) hide)
+    )
+  )
+  (global_label "VCC" (shape input) (at 114.3 111.76 180) (fields_autoplaced)
+    (effects (font (size 1.27 1.27)) (justify right))
+    (property "Intersheet References" "${INTERSHEET_REFS}" (id 0) (at 108.3472 111.6806 0)
+      (effects (font (size 1.27 1.27)) (justify right) hide)
+    )
+  )
+  (global_label "5V" (shape input) (at 138.43 111.76 0) (fields_autoplaced)
+    (effects (font (size 1.27 1.27)) (justify left))
+    (property "Intersheet References" "${INTERSHEET_REFS}" (id 0) (at 143.0523 111.6806 0)
+      (effects (font (size 1.27 1.27)) (justify left) hide)
     )
   )
@@
     (property "Intersheet References" "${INTERSHEET_REFS}" (id 0) (at 57.785 40.64 0)
       (effects (font (size 1.27 1.27)) hide)
+    )
+  )
+  (global_label "VCC" (shape input) (at 76.708 111.76 180) (fields_autoplaced)
+    (effects (font (size 1.27 1.27)) (justify right))
+    (property "Intersheet References" "${INTERSHEET_REFS}" (id 0) (at 70.7552 111.6806 0)
+      (effects (font (size 1.27 1.27)) (justify right) hide)
+    )
+  )
+  (global_label "3V3D" (shape input) (at 100.838 111.76 0) (fields_autoplaced)
+    (effects (font (size 1.27 1.27)) (justify left))
+    (property "Intersheet References" "${INTERSHEET_REFS}" (id 0) (at 107.9398 111.6806 0)
+      (effects (font (size 1.27 1.27)) (justify left) hide)
     )
   )
@@
     (pin "2")
   )
+  (symbol (lib_id "power:GND") (at 126.746 120.904 0) (unit 1)
+    (in_bom yes) (on_board yes)
+    (property "Reference" "#PWR0102" (id 0) (at 126.746 127.254 0)
+      (effects (font (size 1.27 1.27)) hide)
+    )
+    (property "Value" "GND" (id 1) (at 126.873 125.2982 0))
+    (property "Footprint" "" (id 2) (at 126.746 120.904 0)
+      (effects (font (size 1.27 1.27)) hide)
+    )
+    (property "Datasheet" "" (id 3) (at 126.746 120.904 0)
+      (effects (font (size 1.27 1.27)) hide)
+    )
+    (pin "1")
+  )
   (symbol (lib_id "Jumper:Jumper_3_Open") (at 132.08 72.39 270) (unit 1)
     (in_bom yes) (on_board yes) (fields_autoplaced)
@@
     (pin "2")
   )
+  (symbol (lib_id "power:GND") (at 89.154 120.904 0) (unit 1)
+    (in_bom yes) (on_board yes)
+    (property "Reference" "#PWR0106" (id 0) (at 89.154 127.254 0)
+      (effects (font (size 1.27 1.27)) hide)
+    )
+    (property "Value" "GND" (id 1) (at 89.281 125.2982 0))
+    (property "Footprint" "" (id 2) (at 89.154 120.904 0)
+      (effects (font (size 1.27 1.27)) hide)
+    )
+    (property "Datasheet" "" (id 3) (at 89.154 120.904 0)
+      (effects (font (size 1.27 1.27)) hide)
+    )
+    (pin "1")
+  )
   (symbol (lib_id "power:GND") (at 49.53 57.15 0) (unit 1)
     (in_bom yes) (on_board yes)
@@
     (pin "1")
     (pin "2")
+  )
+  (symbol (lib_id "Regulator_Linear:LD1086DTTR") (at 126.746 111.76 0) (unit 1)
+    (in_bom yes) (on_board yes) (fields_autoplaced)
+    (property "Reference" "U7" (id 0) (at 126.746 102.9802 0))
+    (property "Value" "LD1086DTTR" (id 1) (at 126.746 105.5171 0))
+    (property "Footprint" "Package_TO_SOT_SMD:SOT-223" (id 2) (at 126.746 99.06 0)
+      (effects (font (size 1.27 1.27)) hide)
+    )
+    (property "Datasheet" "https://www.st.com/resource/en/datasheet/ld1086.pdf" (id 3) (at 126.746 99.06 0)
+      (effects (font (size 1.27 1.27)) hide)
+    )
+    (pin "1")
+    (pin "2")
+    (pin "3")
   )
   (symbol (lib_id "Device:C") (at 175.895 121.92 0) (unit 1)
@@
     (pin "2")
   )
+  (symbol (lib_id "Regulator_Linear:LD1086DTTR") (at 89.154 111.76 0) (unit 1)
+    (in_bom yes) (on_board yes) (fields_autoplaced)
+    (property "Reference" "U12" (id 0) (at 89.154 102.9802 0))
+    (property "Value" "LD1086DTTR" (id 1) (at 89.154 105.5171 0))
+    (property "Footprint" "Package_TO_SOT_SMD:SOT-223" (id 2) (at 89.154 99.06 0)
+      (effects (font (size 1.27 1.27)) hide)
+    )
+    (property "Datasheet" "https://www.st.com/resource/en/datasheet/ld1086.pdf" (id 3) (at 89.154 99.06 0)
+      (effects (font (size 1.27 1.27)) hide)
+    )
+    (pin "1")
+    (pin "2")
+    (pin "3")
+  )
 )
