File: kicad/NinjaLite/batch03/main-pdb/qLAMP-main.kicad_pcb (KiCad board)
At the start: 2 copper layers, 142 x 58 mm, 118 parts, among them J1 ALI_USB, J13 Conn_01x01_Male, J16 Conn_01x01_Male, J2 Barrel_Jack_Switch, J23 Conn_01x01_Male, J24 Conn_01x02_Male, J25 Conn_01x02_Male, J26 Conn_01x02_Male, J27 Conn_01x02_Male, J3 Conn_01x07_Male, J4 Conn_01x02_Male, J5 Conn_01x01_Male, J6 Conn_01x01_Male, J7 Conn_01x01_Male, Q1 Q_NMOS_GSD, Q3 Q_NMOS_GSD, Q5 Q_NMOS_GSD, U1 NAU7802, U10 TLC5929, U11 IP2721, U14 TCR3DF33,LM(CT, U17 LITE_LCD, U19 CD74HC4067M96, U2 NAU7802, U3 BD433M5FP-CE2, U4 LMP7717MF_NOPB, U5 ESP32-WROOM-32, U6 BA178M05FP-E2, U8 TS12A12511DCNR, U9 SN74LV4051A

Commit message: batch03 finished
Routing:
- net GNDA: vias 248 -> 247
Other:
- board text added: "batch03/main-pdb"
- board text removed: "batch03/main"

Commit message: add reg alt
Parts:
- added U12: LD1086DTTR, Package_TO_SOT_SMD:SOT-223, F.Cu at (174.3, 111.9)
- added U7: LD1086DTTR, Package_TO_SOT_SMD:SOT-223, F.Cu at (172.5, 94.7)
- moved R8 5.71 mm to (181.4, 97.3), turned to 0 degrees
- moved C27 5.67 mm to (175.3, 88.5), turned to -90 degrees
- moved C23 4.21 mm to (180.4, 91.8)
- moved R6 2.31 mm to (184.4, 97.3), turned to 0 degrees
- moved C25 1.79 mm to (172.1, 88.5)
- moved Q3 1.33 mm to (186.1, 93.8)
Routing:
- net 5V: track 242.7 -> 271.0 mm, vias 2 -> 4
- net GNDD: track 346.6 -> 325.2 mm, vias 245 -> 234
- net 3V3D: track 285.4 -> 290.8 mm
- net VCC: track 416.9 -> 412.9 mm
- net /LID_HEATER: track 12.7 -> 8.68 mm
- net Net-(Q3-Pad1): track 3.11 -> 6.60 mm

Commit message: wiring batch04/main
Other:
- board text added: "V(IC,SEL,SELP) must be one of them. V(IP2721|IP2721_D,High,Floating)=20 V(IP2721|IP2721_D,F,F)=15 V(IP2721|IP2721_D,Low,F)=5 V(IP2721_D,F,H)=12 V(IP2721_D,F,L)=9 V(IP2721_MAX12,H,F)=12 V(IP2721_MAX12,F,F)=9 V(IP2721_MAX12,L,F)=5"
Changed lines of the file:
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@@
     (effects (font (size 1 1) (thickness 0.15)))
+  )
+  (gr_text "V(IC,SEL,SELP) must be one of them.\nV(IP2721|IP2721_D,High,Floating)=20\nV(IP2721|IP2721_D,F,F)=15\nV(IP2721|IP2721_D,Low,F)=5\nV(IP2721_D,F,H)=12\nV(IP2721_D,F,L)=9\nV(IP2721_MAX12,H,F)=12\nV(IP2721_MAX12,F,F)=9\nV(IP2721_MAX12,L,F)=5" (at 177.49 61.37) (layer "F.SilkS")
+    (effects (font (size 1 1) (thickness 0.25)) (justify left))
   )
   (gr_text "Personal qLAMP" (at 121.92 123.420016) (layer "F.SilkS")
