File: kicad/NinjaLite/batch04/main/filePhotoMUX.kicad_sch (KiCad schematic)
At the start: 20 parts, among them U19 CD74HC4067M96

Commit message: wiring batch04/main
Parts:
- U19: footprint Package_SO:SSOP-24_5.3x8.2mm_P0.65mm -> Ninja-qPCR:SSOP-24_5.3x8.2mm_P0.65mm-0.83mil
Changed lines of the file:
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@@
       (effects (font (size 1.524 1.524)))
     )
-    (property "Footprint" "Package_SO:SSOP-24_5.3x8.2mm_P0.65mm" (id 2) (at 64.77 127.254 0)
+    (property "Footprint" "Ninja-qPCR:SSOP-24_5.3x8.2mm_P0.65mm-0.83mil" (id 2) (at 64.77 127.254 0)
       (effects (font (size 1.524 1.524)) hide)
     )
@@
       (effects (font (size 1.524 1.524)))
     )
-    (property "Footprint" "Package_SO:SSOP-24_5.3x8.2mm_P0.65mm" (id 2) (at 66.04 49.784 0)
+    (property "Footprint" "Ninja-qPCR:SSOP-24_5.3x8.2mm_P0.65mm-0.83mil" (id 2) (at 66.04 49.784 0)
       (effects (font (size 1.524 1.524)) hide)
     )
