File: kicad/NinjaLite/batch04/main/qLAMP-main.kicad_pcb (KiCad board)
At the start: 2 copper layers, 142 x 58 mm, 99 parts, among them J1 ALI_USB, J13 Conn_01x01_Male, J16 Conn_01x01_Male, J2 Barrel_Jack_Switch, J24 Conn_01x02_Male, J25 Conn_01x02_Male, J3 Conn_01x07_Male, J4 Conn_01x02_Male, J5 Conn_01x01_Male, Q1 Q_NMOS_GSD, Q3 Q_NMOS_GSD, Q5 Q_NMOS_GSD, U1 NAU7802, U10 TLC5929, U11 IP2721, U14 TCR3DF33,LM(CT, U17 LITE_LCD, U19 CD74HC4067M96, U2 NAU7802, U3 BD433M5FP-CE2, U4 LMP7717MF_NOPB, U5 ESP32-WROOM-32, U6 BA178M05FP-E2, U8 TS12A12511DCNR, U9 SN74LV4051A

Commit message: wiring batch04/main
Parts:
- TEXT1, TEXT2, TEXT3: footprint Pin_Headers:Pin_Header_Straight_1x02_Pitch1.27mm -> Pin_Headers:Pin_Header_Straight_1x02_Pitch2.54mm
- moved TWELL1 9.43 mm to (156.3, 92.2), turned to 180 degrees
- moved TLID1 8.68 mm to (167.7, 83.6), turned to 180 degrees
- moved TEXT3 5.63 mm to (159.5, 83.6)
- moved R8 5.54 mm to (183.4, 98.2), turned to -90 degrees
- moved TEXT1 5.29 mm to (164.9, 83.6)
- moved C23 4.46 mm to (180.7, 91.8)
- moved U8 4.45 mm to (158.6, 96.4)
- moved U9 4.41 mm to (165.8, 91.8)
- moved C25 4.40 mm to (174.7, 88.5)
- moved C27 4.22 mm to (174.7, 91.2)
- moved R6 3.49 mm to (185.2, 98.2)
- moved U6 3.39 mm to (176.8, 82.9)
- moved C29 3.27 mm to (185.1, 83.0)
- moved C32 3.27 mm to (184.9, 79.9)
- moved TAIR1 3.02 mm to (159.0, 92.2)
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Connections:
- U9 pad 12: THERM_EXT1 -> THERM_LID
- U9 pad 15: THERM_LID -> THERM_EXT1
Routing:
- net MUX_S2: track 85.5 -> 139.5 mm
- net MUX_S0: track 88.0 -> 141.9 mm
- net MUX_S1: track 89.8 -> 143.7 mm
- net 5V: track 66.8 -> 117.6 mm, vias 2 -> 3
- net THERM_R_SWITCH: track 0.00 -> 48.7 mm
- net GNDA: track 22.1 -> 66.1 mm, vias 5 -> 6
- net THERM_MUX_OUT: track 63.5 -> 99.7 mm
- net /PhotoLED/S_LED_OUT1: track 57.5 -> 31.2 mm
- net /PhotoLED/S_LED_OUT2: track 54.9 -> 28.9 mm
- net /PhotoLED/S_LED_OUT3: track 52.3 -> 26.6 mm
- net THERM_LID: track 0.00 -> 25.4 mm
- net /PhotoLED/S_LED_OUT4: track 49.6 -> 24.4 mm
- net /PhotoLED/S_LED_OUT5: track 47.0 -> 22.1 mm
- net /PhotoLED/S_LED_OUT8: track 39.2 -> 15.3 mm
- net /PhotoLED/S_LED_OUT6: track 44.4 -> 20.6 mm
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Other:
- board text added: "EXT3/2/1"
- board text removed: "EXT1/2/3"

Commit message: wiring batch04/main
Parts:
- moved R22 11.3 mm to (173.3, 115.1)
- moved R21 11.3 mm to (175.1, 115.1)
- moved R23 11.3 mm to (176.9, 115.1)
- moved C11 4.91 mm to (184.4, 124.4), turned to 0 degrees
- moved R12 4.15 mm to (175.2, 117.5)
- moved R19 3.56 mm to (183.4, 98.2)
- moved R8 3.56 mm to (179.9, 98.2)
- moved R20 3.56 mm to (185.2, 98.2)
- moved R6 3.56 mm to (181.6, 98.2)
- moved JP1 1.75 mm to (147.0, 126.0)
Connections:
- R12 pad 1: SD_CD -> 3V3D
- R12 pad 2: 3V3D -> TACT1
- R21 pad 1: TACT2 -> TACT3
- R22 pad 1: TACT3 -> TACT2
- R23 pad 2: TACT1 -> SD_CD
- U17 pad 1: SD_CD -> TACT3
- U17 pad 2: SD_CS -> TACT2
- U17 pad 3: MOSI -> TACT1
- U17 pad 4: MISO -> SD_CD
- U17 pad 5: TACT3 -> SD_CS
- U17 pad 6: TACT2 -> SCLK
- U17 pad 7: TACT1 -> MISO
- U17 pad 8: SCLK -> MOSI
- U5 pad 24: TACT3 -> TACT2
- U5 pad 25: TACT2 -> TACT3
- U5 pad 28: SD_CD -> Net-(J5-Pad1)
- U5 pad 7: TACT1 -> SD_CD
- U5 pad 9: Net-(J5-Pad1) -> TACT1
Routing:
- net 5V: track 117.6 -> 200.6 mm, vias 3 -> 4
- net /PhotoLED/S_LED_OUT1: track 31.2 -> 58.9 mm
- net /PhotoLED/S_LED_OUT2: track 28.9 -> 56.3 mm
- net /PhotoLED/S_LED_OUT3: track 26.6 -> 53.6 mm
- net /PhotoLED/S_LED_OUT4: track 24.4 -> 51.0 mm
- net /PhotoLED/S_LED_OUT5: track 22.1 -> 48.4 mm
- net /PhotoLED/S_LED_OUT6: track 20.6 -> 46.6 mm
- net /PhotoLED/S_LED_OUT7: track 17.6 -> 43.2 mm
- net I2C_SCL: track 84.8 -> 110.4 mm, vias 1 -> 2
- net /PhotoLED/S_LED_OUT8: track 15.3 -> 40.6 mm
- net 3V3D: track 120.2 -> 144.7 mm, vias 3 -> 5
- net I2C_SDA: track 83.7 -> 107.0 mm, vias 1 -> 2
- net MOSI: track 38.9 -> 55.9 mm, vias 1 -> 2
- net MUX_S2: track 139.5 -> 155.5 mm, vias 1 -> 2
- net LED_BLANK: track 43.0 -> 58.3 mm
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
Commit message: ordered batch04
Parts:
- moved R12 19.2 mm to (181.7, 99.4)
- moved R23 17.4 mm to (184.4, 99.4), turned to 0 degrees
- moved R22 16.7 mm to (179.1, 99.4), turned to 180 degrees
- moved R21 15.8 mm to (176.4, 99.4), turned to 180 degrees
- moved U3 8.04 mm to (168.2, 102.7)
- moved J5 6.47 mm to (188.6, 120.7)
- moved C28 3.77 mm to (163.1, 101.2), turned to -90 degrees
- moved R20 3.55 mm to (181.7, 97.4), turned to 180 degrees
- moved R8 3.55 mm to (176.4, 97.4), turned to 0 degrees
- moved C31 3.48 mm to (160.6, 101.8), turned to -90 degrees
- moved C27 3.21 mm to (175.7, 88.2), turned to 90 degrees
- moved R6 2.69 mm to (179.1, 97.4), turned to 0 degrees
- moved C25 1.57 mm to (173.2, 89.0), turned to 90 degrees
- moved R19 1.28 mm to (184.4, 97.4), turned to 180 degrees
- moved Q5 0.76 mm to (199.4, 93.6)
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Routing:
- net GNDD: track 74.0 -> 370.9 mm, vias 5 -> 226
- net 3V3D: track 144.7 -> 255.6 mm, vias 5 -> 12
- net NAU_DRDY: track 95.3 -> 152.1 mm, vias 1 -> 2
- net TACT2: track 0.00 -> 53.2 mm, vias 0 -> 3
- net THERM_R_SWITCH: track 57.0 -> 106.8 mm, vias 1 -> 2
- net I2C_SCL: track 110.4 -> 154.9 mm, vias 2 -> 3
- net LED_LAT: track 48.8 -> 92.1 mm, vias 1 -> 2
- net MUX_S2: track 155.5 -> 196.4 mm, vias 2 -> 3
- net TACT3: track 0.00 -> 40.2 mm, vias 0 -> 2
- net VCC: track 52.6 -> 92.4 mm
- net MUX_S1: track 158.0 -> 197.6 mm, vias 2 -> 3
- net I2C_SDA: track 107.0 -> 144.8 mm, vias 2 -> 3
- net 5V: track 200.6 -> 237.7 mm
- net MOSI: track 55.9 -> 87.6 mm, vias 2 -> 4
- net MUX_S3: track 107.2 -> 136.1 mm, vias 1 -> 2
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Other:
- board text removed: "J26"
- board text removed: "LPF_OUT"
