File: kicad/NinjaLite/batch04/lcd/qLAMP-lcd.kicad_sch (KiCad schematic)
At the start: 13 parts, among them J1 Conn_01x04_Male, J2 Conn_01x04_Male, J3 Conn_01x04_Male, J4 ALI_Micro_SD_Card, SW1 TACTILE_4, SW2 TACTILE_4, SW3 TACTILE_4

Commit message: ordered batch04
Parts:
- D2: footprint Ninja-qPCR:I2C_SSD1306_LCD -> Ninja-qPCR:ALI_I2C_LCD
Connections:
- net MISO: now also J2.3 (Pin_3); no longer J1.4 (Pin_4)
- net MOSI: now also J2.4 (Pin_4); no longer J1.3 (Pin_3)
- net SCLK: now also J2.2 (Pin_2); no longer J2.4 (Pin_4)
- net SD_CD: now also J1.4 (Pin_4); no longer J1.1 (Pin_1)
- net SD_CS: now also J2.1 (Pin_1); no longer J1.2 (Pin_2)
- net TACT1: now also J1.3 (Pin_3); no longer J2.3 (Pin_3)
- net TACT2: now also J1.2 (Pin_2); no longer J2.2 (Pin_2)
- net TACT3: now also J1.1 (Pin_1); no longer J2.1 (Pin_1)
- net SCL renamed I2C_SCL
- net SDA renamed I2C_SDA
- no-connect marks 2 -> 3
Other:
- moved on the sheet: J4
Changed lines of the file:
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@@
   (junction (at 183.388 127.508) (diameter 0) (color 0 0 0 0)
   )
+  (no_connect (at 221.234 67.056))
   (no_connect (at 172.974 46.736))
   (no_connect (at 172.974 64.516))
@@
     (stroke (width 0) (type default) (color 0 0 0 0))
   )
-  (global_label "TACT3" (shape input) (at 74.168 55.626 180) (fields_autoplaced)
-    (effects (font (size 1.27 1.27)) (justify right))
-    (property "Intersheet References" "${INTERSHEET_REFS}" (id 0) (at 66.3405 55.5466 0)
-      (effects (font (size 1.27 1.27)) (justify right) hide)
-    )
-  )
-  (global_label "TACT1" (shape input) (at 74.168 60.706 180) (fields_autoplaced)
-    (effects (font (size 1.27 1.27)) (justify right))
-    (property "Intersheet References" "${INTERSHEET_REFS}" (id 0) (at 66.3405 60.6266 0)
+  (global_label "TACT3" (shape input) (at 74.168 40.386 180) (fields_autoplaced)
+    (effects (font (size 1.27 1.27)) (justify right))
+    (property "Intersheet References" "${INTERSHEET_REFS}" (id 0) (at 66.3405 40.3066 0)
+      (effects (font (size 1.27 1.27)) (justify right) hide)
+    )
+  )
+  (global_label "TACT1" (shape input) (at 74.168 45.466 180) (fields_autoplaced)
+    (effects (font (size 1.27 1.27)) (justify right))
+    (property "Intersheet References" "${INTERSHEET_REFS}" (id 0) (at 66.3405 45.3866 0)
       (effects (font (size 1.27 1.27)) (justify right) hide)
     )
@@
     )
   )
-  (global_label "SDA" (shape input) (at 70.104 132.588 180) (fields_autoplaced)
-    (effects (font (size 1.27 1.27)) (justify right))
-    (property "Intersheet References" "${INTERSHEET_REFS}" (id 0) (at 64.2117 132.5086 0)
+  (global_label "I2C_SDA" (shape input) (at 70.104 132.588 180) (fields_autoplaced)
+    (effects (font (size 1.27 1.27)) (justify right))
+    (property "Intersheet References" "${INTERSHEET_REFS}" (id 0) (at 60.1598 132.5086 0)
       (effects (font (size 1.27 1.27)) (justify right) hide)
     )
@@
     )
   )
-  (global_label "SCL" (shape input) (at 74.168 73.406 180) (fields_autoplaced)
-    (effects (font (size 1.27 1.27)) (justify right))
-    (property "Intersheet References" "${INTERSHEET_REFS}" (id 0) (at 68.3362 73.3266 0)
+  (global_label "I2C_SCL" (shape input) (at 74.168 73.406 180) (fields_autoplaced)
+    (effects (font (size 1.27 1.27)) (justify right))
+    (property "Intersheet References" "${INTERSHEET_REFS}" (id 0) (at 64.2843 73.3266 0)
       (effects (font (size 1.27 1.27)) (justify right) hide)
     )
@@
     )
   )
-  (global_label "MISO" (shape input) (at 74.168 48.006 180) (fields_autoplaced)
-    (effects (font (size 1.27 1.27)) (justify right))
-    (property "Intersheet References" "${INTERSHEET_REFS}" (id 0) (at 67.2476 47.9266 0)
+  (global_label "MISO" (shape input) (at 74.168 60.706 180) (fields_autoplaced)
+    (effects (font (size 1.27 1.27)) (justify right))
+    (property "Intersheet References" "${INTERSHEET_REFS}" (id 0) (at 67.2476 60.6266 0)
       (effects (font (size 1.27 1.27)) (justify right) hide)
     )
@@
     )
   )
-  (global_label "SD_CD" (shape input) (at 74.168 40.386 180) (fields_autoplaced)
-    (effects (font (size 1.27 1.27)) (justify right))
-    (property "Intersheet References" "${INTERSHEET_REFS}" (id 0) (at 65.8567 40.3066 0)
+  (global_label "SD_CD" (shape input) (at 74.168 48.006 180) (fields_autoplaced)
+    (effects (font (size 1.27 1.27)) (justify right))
+    (property "Intersheet References" "${INTERSHEET_REFS}" (id 0) (at 65.8567 47.9266 0)
       (effects (font (size 1.27 1.27)) (justify right) hide)
     )
@@
     )
   )
-  (global_label "SD_CS" (shape input) (at 74.168 42.926 180) (fields_autoplaced)
-    (effects (font (size 1.27 1.27)) (justify right))
-    (property "Intersheet References" "${INTERSHEET_REFS}" (id 0) (at 65.9171 42.8466 0)
-      (effects (font (size 1.27 1.27)) (justify right) hide)
-    )
-  )
-  (global_label "SCL" (shape input) (at 70.104 130.048 180) (fields_autoplaced)
-    (effects (font (size 1.27 1.27)) (justify right))
-    (property "Intersheet References" "${INTERSHEET_REFS}" (id 0) (at 64.2722 129.9686 0)
+  (global_label "SD_CS" (shape input) (at 74.168 55.626 180) (fields_autoplaced)
+    (effects (font (size 1.27 1.27)) (justify right))
+    (property "Intersheet References" "${INTERSHEET_REFS}" (id 0) (at 65.9171 55.5466 0)
+      (effects (font (size 1.27 1.27)) (justify right) hide)
+    )
+  )
+  (global_label "I2C_SCL" (shape input) (at 70.104 130.048 180) (fields_autoplaced)
+    (effects (font (size 1.27 1.27)) (justify right))
+    (property "Intersheet References" "${INTERSHEET_REFS}" (id 0) (at 60.2203 129.9686 0)
       (effects (font (size 1.27 1.27)) (justify right) hide)
     )
@@
     )
   )
-  (global_label "SDA" (shape input) (at 74.168 75.946 180) (fields_autoplaced)
-    (effects (font (size 1.27 1.27)) (justify right))
-    (property "Intersheet References" "${INTERSHEET_REFS}" (id 0) (at 68.2757 75.8666 0)
+  (global_label "I2C_SDA" (shape input) (at 74.168 75.946 180) (fields_autoplaced)
+    (effects (font (size 1.27 1.27)) (justify right))
+    (property "Intersheet References" "${INTERSHEET_REFS}" (id 0) (at 64.2238 75.8666 0)
       (effects (font (size 1.27 1.27)) (justify right) hide)
     )
@@
     )
   )
-  (global_label "MOSI" (shape input) (at 74.168 45.466 180) (fields_autoplaced)
-    (effects (font (size 1.27 1.27)) (justify right))
-    (property "Intersheet References" "${INTERSHEET_REFS}" (id 0) (at 67.2476 45.3866 0)
+  (global_label "MOSI" (shape input) (at 74.168 63.246 180) (fields_autoplaced)
+    (effects (font (size 1.27 1.27)) (justify right))
+    (property "Intersheet References" "${INTERSHEET_REFS}" (id 0) (at 67.2476 63.1666 0)
       (effects (font (size 1.27 1.27)) (justify right) hide)
     )
@@
     )
   )
-  (global_label "SCLK" (shape input) (at 74.168 63.246 180) (fields_autoplaced)
-    (effects (font (size 1.27 1.27)) (justify right))
-    (property "Intersheet References" "${INTERSHEET_REFS}" (id 0) (at 67.0662 63.1666 0)
+  (global_label "SCLK" (shape input) (at 74.168 58.166 180) (fields_autoplaced)
+    (effects (font (size 1.27 1.27)) (justify right))
+    (property "Intersheet References" "${INTERSHEET_REFS}" (id 0) (at 67.0662 58.0866 0)
       (effects (font (size 1.27 1.27)) (justify right) hide)
     )
@@
     )
   )
-  (global_label "TACT2" (shape input) (at 74.168 58.166 180) (fields_autoplaced)
-    (effects (font (size 1.27 1.27)) (justify right))
-    (property "Intersheet References" "${INTERSHEET_REFS}" (id 0) (at 66.3405 58.0866 0)
+  (global_label "TACT2" (shape input) (at 74.168 42.926 180) (fields_autoplaced)
+    (effects (font (size 1.27 1.27)) (justify right))
+    (property "Intersheet References" "${INTERSHEET_REFS}" (id 0) (at 66.3405 42.8466 0)
       (effects (font (size 1.27 1.27)) (justify right) hide)
     )
@@
       (effects (font (size 1.27 1.27)) (justify left))
     )
-    (property "Footprint" "Ninja-qPCR:I2C_SSD1306_LCD" (id 2) (at 91.694 127.508 0)
+    (property "Footprint" "Ninja-qPCR:ALI_I2C_LCD" (id 2) (at 91.694 127.508 0)
       (effects (font (size 1.27 1.27)) hide)
     )
@@
   (symbol_instances
     (path "/cf609d9f-a23f-493e-b93e-9d03f9c0c792"
-      (reference "D2") (unit 1) (value "I2C_SSD1306_LCD") (footprint "Ninja-qPCR:I2C_SSD1306_LCD")
+      (reference "D2") (unit 1) (value "I2C_SSD1306_LCD") (footprint "Ninja-qPCR:ALI_I2C_LCD")
     )
     (path "/cff34e0d-7659-4dfc-9864-1c04d35138d1"
