File: kicad/NinjaLite/batch05/main/filePower.kicad_sch (KiCad schematic)
At the start: 27 parts, among them J1 ALI_USB, J2 Barrel_Jack_Switch, Q1 Q_NMOS_GSD, U11 IP2721, U14 TCR3DF33,LM(CT, U3 BD433M5FP-CE2, U6 BA178M05FP-E2

Commit message: autodeploy
Parts:
- added U7: BD433M5FP-CE2, Ninja-qPCR:REG_TO252-3-INV, symbol Ninja-qPCR:REG_TO252-3
Connections:
- net 3V3D: now also U7.2 (VOUT)
- net GND: now also U7.3 (GND)
- net VCC: now also U7.1 (VIN)
Changed lines of the file:
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@@
+    (stroke (width 0) (type default) (color 0 0 0 0))
+  )
+  (wire (pts (xy 240.284 24.13) (xy 242.824 24.13))
     (stroke (width 0) (type default) (color 0 0 0 0))
   )
@@
     (stroke (width 0) (type default) (color 0 0 0 0))
   )
+  (wire (pts (xy 260.604 24.13) (xy 263.398 24.13))
+    (stroke (width 0) (type default) (color 0 0 0 0))
+  )
   (wire (pts (xy 124.46 68.58) (xy 124.46 80.01))
     (stroke (width 0) (type default) (color 0 0 0 0))
@@
   )
   (wire (pts (xy 211.455 119.38) (xy 211.455 121.92))
+    (stroke (width 0) (type default) (color 0 0 0 0))
+  )
+  (wire (pts (xy 251.714 31.75) (xy 251.714 34.29))
     (stroke (width 0) (type default) (color 0 0 0 0))
   )
@@
     (effects (font (size 1.27 1.27)) (justify left))
     (property "Intersheet References" "${INTERSHEET_REFS}" (id 0) (at 80.645 -61.595 0)
+      (effects (font (size 1.27 1.27)) hide)
+    )
+  )
+  (global_label "3V3D" (shape input) (at 263.398 24.13 0) (fields_autoplaced)
+    (effects (font (size 1.27 1.27)) (justify left))
+    (property "Intersheet References" "${INTERSHEET_REFS}" (id 0) (at 79.248 -81.28 0)
       (effects (font (size 1.27 1.27)) hide)
     )
@@
     (effects (font (size 1.27 1.27)) (justify right))
     (property "Intersheet References" "${INTERSHEET_REFS}" (id 0) (at 166.8277 111.6806 0)
+      (effects (font (size 1.27 1.27)) (justify right) hide)
+    )
+  )
+  (global_label "VCC" (shape input) (at 240.284 24.13 180) (fields_autoplaced)
+    (effects (font (size 1.27 1.27)) (justify right))
+    (property "Intersheet References" "${INTERSHEET_REFS}" (id 0) (at 234.3312 24.0506 0)
       (effects (font (size 1.27 1.27)) (justify right) hide)
     )
@@
     (pin "2")
   )
+  (symbol (lib_id "power:GND") (at 251.714 34.29 0) (unit 1)
+    (in_bom yes) (on_board yes)
+    (property "Reference" "#PWR0102" (id 0) (at 251.714 40.64 0)
+      (effects (font (size 1.27 1.27)) hide)
+    )
+    (property "Value" "GND" (id 1) (at 251.841 38.6842 0))
+    (property "Footprint" "" (id 2) (at 251.714 34.29 0)
+      (effects (font (size 1.27 1.27)) hide)
+    )
+    (property "Datasheet" "" (id 3) (at 251.714 34.29 0)
+      (effects (font (size 1.27 1.27)) hide)
+    )
+    (pin "1")
+  )
   (symbol (lib_id "Device:R") (at 124.46 49.53 180) (unit 1)
     (in_bom yes) (on_board yes)
@@
     (pin "1")
   )
+  (symbol (lib_id "Ninja-qPCR:REG_TO252-3") (at 251.714 22.86 0) (unit 1)
+    (in_bom yes) (on_board yes)
+    (property "Reference" "U7" (id 0) (at 251.714 19.05 0))
+    (property "Value" "BD433M5FP-CE2" (id 1) (at 252.349 21.59 0))
+    (property "Footprint" "Ninja-qPCR:REG_TO252-3-INV" (id 2) (at 250.444 21.59 0)
+      (effects (font (size 1.27 1.27)) hide)
+    )
+    (property "Datasheet" "" (id 3) (at 250.444 21.59 0)
+      (effects (font (size 1.27 1.27)) hide)
+    )
+    (pin "1")
+    (pin "2")
+    (pin "3")
+  )
   (symbol (lib_id "Jumper:Jumper_3_Open") (at 124.46 62.23 270) (unit 1)
