File: kicad/NinjaLite/batch07/connector/qLAMP-connector.kicad_pcb (KiCad board)
At the start: 2 copper layers, 76 x 36 mm, 5 parts, among them J1 Conn_01x07_Male, J2 Conn_01x07_Male, J3 Conn_01x04_Male, J4 Conn_01x04_Male, J5 Conn_01x14_Male

Commit message: sync
Parts:
- removed J5: Conn_01x14_Male, Connector_PinSocket_2.54mm:PinSocket_1x14_P2.54mm_Vertical
- J1: value Conn_01x07_Male -> Conn_01x18_Male; footprint Connector_PinSocket_2.54mm:PinSocket_1x07_P2.54mm_Vertical -> Connector_PinSocket_2.54mm:PinSocket_2x09_P2.54mm_Vertical
- J2: value Conn_01x07_Male -> Conn_01x14_Male; footprint Connector_PinSocket_2.54mm:PinSocket_1x07_P2.54mm_Vertical -> Connector_PinSocket_2.54mm:PinSocket_1x14_P2.54mm_Vertical
- J4: value Conn_01x04_Male -> Conn_01x18_Male; footprint Connector_PinSocket_2.54mm:PinSocket_1x04_P2.54mm_Vertical -> Connector_PinSocket_1.27mm:PinSocket_2x09_P1.27mm_Vertical
- moved J3 73.4 mm to (216.0, 107.3)
- moved J4 63.4 mm to (144.9, 109.6)
- moved J2 11.4 mm to (135.0, 120.0)
- moved J1 3.04 mm to (138.7, 112.7)
Connections:
- J1 pad 1: Net-(J1-Pad1) -> Net-(J2-Pad1)
- J1 pad 2: Net-(J1-Pad2) -> Net-(J2-Pad2)
- J1 pad 3: Net-(J1-Pad3) -> Net-(J2-Pad3)
- J1 pad 4: Net-(J1-Pad4) -> Net-(J2-Pad4)
- J1 pad 5: Net-(J1-Pad5) -> Net-(J2-Pad5)
- J1 pad 6: Net-(J1-Pad6) -> Net-(J2-Pad6)
- J1 pad 7: Net-(J1-Pad7) -> Net-(J2-Pad7)
- J4 pad 1: Net-(J3-Pad1) -> unconnected-(J4-Pad1)
- J4 pad 2: Net-(J3-Pad2) -> unconnected-(J4-Pad2)
- J4 pad 3: Net-(J3-Pad3) -> unconnected-(J4-Pad3)
- J4 pad 4: Net-(J3-Pad4) -> unconnected-(J4-Pad4)
Routing:
- added copper zone on B.Cu, net unconnected-(J4-Pad12)
- added copper zone on F.Cu, net unconnected-(J4-Pad12)
- removed copper zone on B.Cu, net (none)
- removed copper zone on F.Cu, net (none)
Other:
- board size 76 x 36 mm -> 84 x 36 mm
- board text added: "84x36mm"
- board text removed: "76x36mm"
