File: kicad/NinjaLite/batch07/connector/qLAMP-connector.kicad_sch (KiCad schematic)
At the start: 5 parts, among them J1 Conn_01x07_Male, J2 Conn_01x07_Male, J3 Conn_01x04_Male, J4 Conn_01x04_Male, J5 Conn_01x14_Male

Commit message: sync
Parts:
- removed J1, J2: Conn_01x07_Male, Connector_PinSocket_2.54mm:PinSocket_1x07_P2.54mm_Vertical, symbol Connector:Conn_01x07_Male
- removed J3: Conn_01x04_Male, Connector_PinSocket_2.54mm:PinSocket_1x04_P2.54mm_Vertical, symbol Connector:Conn_01x04_Male
- added J1: Conn_01x18_Male, Connector_PinSocket_2.54mm:PinSocket_2x09_P2.54mm_Vertical, symbol Connector:Conn_01x18_Male
- added J4: Conn_01x18_Male, Connector_PinSocket_1.27mm:PinSocket_2x09_P1.27mm_Vertical, symbol Connector:Conn_01x18_Male
- renumbered J5 to J2, J4 to J3
Connections:
- net at J2.1 (Pin_1): now also J1.1 (Pin_1)
- net at J2.10 (Pin_10): now also J1.10 (Pin_10)
- net at J2.11 (Pin_11): now also J1.11 (Pin_11)
- net at J2.12 (Pin_12): now also J1.12 (Pin_12)
- net at J2.13 (Pin_13): now also J1.13 (Pin_13)
- net at J2.14 (Pin_14): now also J1.14 (Pin_14)
- net at J2.2 (Pin_2): now also J1.2 (Pin_2)
- net at J2.3 (Pin_3): now also J1.3 (Pin_3)
- net at J2.4 (Pin_4): now also J1.4 (Pin_4)
- net at J2.5 (Pin_5): now also J1.5 (Pin_5)
- net at J2.6 (Pin_6): now also J1.6 (Pin_6)
- net at J2.7 (Pin_7): now also J1.7 (Pin_7)
- net at J2.8 (Pin_8): now also J1.8 (Pin_8)
- net at J2.9 (Pin_9): now also J1.9 (Pin_9)
- net at J3.1 (Pin_1): now also J1.15 (Pin_15)
- net at J3.2 (Pin_2): now also J1.16 (Pin_16)
- net at J3.3 (Pin_3): now also J1.17 (Pin_17)
- net at J3.4 (Pin_4): now also J1.18 (Pin_18)
Other:
- moved on the sheet: J2, J3
