File: kicad/NinjaLite/batch07/main/filePhotoLED.kicad_sch (KiCad schematic)
At the start: 6 parts, among them U10 TLC5929

Commit message: wiring batch7
Parts:
- JLN1, JLS1: footprint Connector_PinSocket_1.27mm:PinSocket_2x05_P1.27mm_Vertical -> Connector_PinSocket_1.27mm:PinSocket_2x05_P1.27mm_Vertical_SMD
Changed lines of the file:
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@@
       (effects (font (size 1.27 1.27)))
     )
-    (property "Footprint" "Connector_PinSocket_1.27mm:PinSocket_2x05_P1.27mm_Vertical" (at 220.98 68.58 0)
+    (property "Footprint" "Connector_PinSocket_1.27mm:PinSocket_2x05_P1.27mm_Vertical_SMD" (at 220.98 68.58 0)
       (effects (font (size 1.27 1.27)) hide)
     )
@@
       (effects (font (size 1.27 1.27)) (justify right))
     )
-    (property "Footprint" "Connector_PinSocket_1.27mm:PinSocket_2x05_P1.27mm_Vertical" (at 220.98 119.38 0)
+    (property "Footprint" "Connector_PinSocket_1.27mm:PinSocket_2x05_P1.27mm_Vertical_SMD" (at 220.98 119.38 0)
       (effects (font (size 1.27 1.27)) hide)
     )
