File: kicad/NinjaLite/batch07/main/filePhotoMUX.kicad_sch (KiCad schematic)
At the start: 20 parts, among them U19 CD74HC4067M96

Commit message: wiring batch7
Parts:
- D10A1, D11A1, D12A1, D13A1, D14A1, D15A1, D16A1, D1A1, D2A1, D3A1, D4A1, D5A1, D6A1, D7A1, D8A1, D9A1: footprint Ninja-qPCR:SFH2200_2201_2240 -> Ninja:SFH2200_2201_2240
- U19: footprint Ninja-qPCR:SSOP-24_5.3x8.2mm_P0.65mm-0.83mil -> Ninja:SSOP-24_5.3x8.2mm_P0.65mm-0.83mil
Changed lines of the file:
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@@
       (effects (font (size 1.524 1.524)))
     )
-    (property "Footprint" "Ninja-qPCR:SSOP-24_5.3x8.2mm_P0.65mm-0.83mil" (at 64.77 127.254 0)
+    (property "Footprint" "Ninja:SSOP-24_5.3x8.2mm_P0.65mm-0.83mil" (at 64.77 127.254 0)
       (effects (font (size 1.524 1.524)) hide)
     )
@@
       (effects (font (size 1.524 1.524)))
     )
-    (property "Footprint" "Ninja-qPCR:SSOP-24_5.3x8.2mm_P0.65mm-0.83mil" (at 66.04 49.784 0)
+    (property "Footprint" "Ninja:SSOP-24_5.3x8.2mm_P0.65mm-0.83mil" (at 66.04 49.784 0)
       (effects (font (size 1.524 1.524)) hide)
     )
@@
       (effects (font (size 1.27 1.27)))
     )
-    (property "Footprint" "Ninja-qPCR:SFH2200_2201_2240" (at 186.69 77.47 0)
+    (property "Footprint" "Ninja:SFH2200_2201_2240" (at 186.69 77.47 0)
       (effects (font (size 1.27 1.27)) hide)
     )
@@
       (effects (font (size 1.27 1.27)))
     )
-    (property "Footprint" "Ninja-qPCR:SFH2200_2201_2240" (at 229.87 57.15 0)
+    (property "Footprint" "Ninja:SFH2200_2201_2240" (at 229.87 57.15 0)
       (effects (font (size 1.27 1.27)) hide)
     )
@@
       (effects (font (size 1.27 1.27)))
     )
-    (property "Footprint" "Ninja-qPCR:SFH2200_2201_2240" (at 151.13 97.79 0)
+    (property "Footprint" "Ninja:SFH2200_2201_2240" (at 151.13 97.79 0)
       (effects (font (size 1.27 1.27)) hide)
     )
@@
       (effects (font (size 1.27 1.27)))
     )
-    (property "Footprint" "Ninja-qPCR:SFH2200_2201_2240" (at 265.43 97.79 0)
+    (property "Footprint" "Ninja:SFH2200_2201_2240" (at 265.43 97.79 0)
       (effects (font (size 1.27 1.27)) hide)
     )
@@
       (effects (font (size 1.27 1.27)))
     )
-    (property "Footprint" "Ninja-qPCR:SFH2200_2201_2240" (at 151.13 57.15 0)
+    (property "Footprint" "Ninja:SFH2200_2201_2240" (at 151.13 57.15 0)
       (effects (font (size 1.27 1.27)) hide)
     )
@@
       (effects (font (size 1.27 1.27)))
     )
-    (property "Footprint" "Ninja-qPCR:SFH2200_2201_2240" (at 229.87 118.11 0)
+    (property "Footprint" "Ninja:SFH2200_2201_2240" (at 229.87 118.11 0)
       (effects (font (size 1.27 1.27)) hide)
     )
@@
       (effects (font (size 1.27 1.27)))
     )
-    (property "Footprint" "Ninja-qPCR:SFH2200_2201_2240" (at 265.43 57.15 0)
+    (property "Footprint" "Ninja:SFH2200_2201_2240" (at 265.43 57.15 0)
       (effects (font (size 1.27 1.27)) hide)
     )
@@
       (effects (font (size 1.27 1.27)))
     )
-    (property "Footprint" "Ninja-qPCR:SFH2200_2201_2240" (at 229.87 97.79 0)
+    (property "Footprint" "Ninja:SFH2200_2201_2240" (at 229.87 97.79 0)
       (effects (font (size 1.27 1.27)) hide)
     )
@@
       (effects (font (size 1.27 1.27)))
     )
-    (property "Footprint" "Ninja-qPCR:SFH2200_2201_2240" (at 229.87 77.47 0)
+    (property "Footprint" "Ninja:SFH2200_2201_2240" (at 229.87 77.47 0)
       (effects (font (size 1.27 1.27)) hide)
     )
@@
       (effects (font (size 1.27 1.27)))
     )
-    (property "Footprint" "Ninja-qPCR:SFH2200_2201_2240" (at 151.13 118.11 0)
+    (property "Footprint" "Ninja:SFH2200_2201_2240" (at 151.13 118.11 0)
       (effects (font (size 1.27 1.27)) hide)
     )
@@
       (effects (font (size 1.27 1.27)))
     )
-    (property "Footprint" "Ninja-qPCR:SFH2200_2201_2240" (at 265.43 77.47 0)
+    (property "Footprint" "Ninja:SFH2200_2201_2240" (at 265.43 77.47 0)
       (effects (font (size 1.27 1.27)) hide)
     )
@@
       (effects (font (size 1.27 1.27)))
     )
-    (property "Footprint" "Ninja-qPCR:SFH2200_2201_2240" (at 151.13 77.47 0)
+    (property "Footprint" "Ninja:SFH2200_2201_2240" (at 151.13 77.47 0)
       (effects (font (size 1.27 1.27)) hide)
     )
@@
       (effects (font (size 1.27 1.27)))
     )
-    (property "Footprint" "Ninja-qPCR:SFH2200_2201_2240" (at 186.69 57.15 0)
+    (property "Footprint" "Ninja:SFH2200_2201_2240" (at 186.69 57.15 0)
       (effects (font (size 1.27 1.27)) hide)
     )
@@
       (effects (font (size 1.27 1.27)))
     )
-    (property "Footprint" "Ninja-qPCR:SFH2200_2201_2240" (at 186.69 97.79 0)
+    (property "Footprint" "Ninja:SFH2200_2201_2240" (at 186.69 97.79 0)
       (effects (font (size 1.27 1.27)) hide)
     )
@@
       (effects (font (size 1.27 1.27)))
     )
-    (property "Footprint" "Ninja-qPCR:SFH2200_2201_2240" (at 265.43 118.11 0)
+    (property "Footprint" "Ninja:SFH2200_2201_2240" (at 265.43 118.11 0)
       (effects (font (size 1.27 1.27)) hide)
     )
@@
       (effects (font (size 1.27 1.27)))
     )
-    (property "Footprint" "Ninja-qPCR:SFH2200_2201_2240" (at 186.69 118.11 0)
-      (effects (font (size 1.27 1.27)) hide)
-    )
+    (property "Footprint" "Ninja:SFH2200_2201_2240" (at 186.69 118.11 0)
+      (effects (font (size 1.27 1.27)) hide)
+    )
