File: kicad/NinjaLite/batch07/main/filePhotoThermistors.kicad_sch (KiCad schematic)
At the start: 10 parts, among them U8 TS12A12511DCNR, U9 SN74LV4051A

Commit message: wiring batch7
Parts:
- TEXT1, TEXT2, TEXT3, TLID1, TWELL1: footprint Pin_Headers:Pin_Header_Straight_1x02_Pitch2.54mm -> Connector_PinHeader_2.54mm:PinHeader_1x02_P2.54mm_Vertical
- U8: footprint Ninja-qPCR:SOT-23-8-8.3mil -> Ninja:SOT-23-8-8.3mil
Changed lines of the file:
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@@
       (effects (font (size 1.524 1.524)))
     )
-    (property "Footprint" "Ninja-qPCR:SOT-23-8-8.3mil" (at 64.77 85.344 0)
+    (property "Footprint" "Ninja:SOT-23-8-8.3mil" (at 64.77 85.344 0)
       (effects (font (size 1.524 1.524)) hide)
     )
@@
       (effects (font (size 1.27 1.27)))
     )
-    (property "Footprint" "Pin_Headers:Pin_Header_Straight_1x02_Pitch2.54mm" (at 254 80.01 0)
+    (property "Footprint" "Connector_PinHeader_2.54mm:PinHeader_1x02_P2.54mm_Vertical" (at 254 80.01 0)
       (effects (font (size 1.27 1.27)) hide)
     )
@@
       (effects (font (size 1.27 1.27)))
     )
-    (property "Footprint" "Pin_Headers:Pin_Header_Straight_1x02_Pitch2.54mm" (at 254 64.77 0)
+    (property "Footprint" "Connector_PinHeader_2.54mm:PinHeader_1x02_P2.54mm_Vertical" (at 254 64.77 0)
       (effects (font (size 1.27 1.27)) hide)
     )
@@
       (effects (font (size 1.27 1.27)))
     )
-    (property "Footprint" "Pin_Headers:Pin_Header_Straight_1x02_Pitch2.54mm" (at 254 88.9 0)
+    (property "Footprint" "Connector_PinHeader_2.54mm:PinHeader_1x02_P2.54mm_Vertical" (at 254 88.9 0)
       (effects (font (size 1.27 1.27)) hide)
     )
@@
       (effects (font (size 1.27 1.27)))
     )
-    (property "Footprint" "Pin_Headers:Pin_Header_Straight_1x02_Pitch2.54mm" (at 254 49.53 0)
+    (property "Footprint" "Connector_PinHeader_2.54mm:PinHeader_1x02_P2.54mm_Vertical" (at 254 49.53 0)
       (effects (font (size 1.27 1.27)) hide)
     )
@@
       (effects (font (size 1.27 1.27)))
     )
-    (property "Footprint" "Pin_Headers:Pin_Header_Straight_1x02_Pitch2.54mm" (at 254 96.52 0)
-      (effects (font (size 1.27 1.27)) hide)
-    )
+    (property "Footprint" "Connector_PinHeader_2.54mm:PinHeader_1x02_P2.54mm_Vertical" (at 254 96.52 0)
+      (effects (font (size 1.27 1.27)) hide)
+    )
